File: schematics/power_switch.kicad_sch (KiCad schematic)
At the start: 19 parts, among them J1 XT90PW-M, Q1 PSMN3R7-100BSEJ, Q2 PSMN3R7-100BSEJ, Q3 PSMN3R7-100BSEJ, Q4 PSMN3R7-100BSEJ, Q5 PSMN3R7-100BSEJ, SW1 SW_SPST, U1 TPS2490

Commit message: fixed footprints
Parts:
- J1: symbol xt90:XT90PW-M -> XT90PW-M:XT90PW-M
- Q1, Q2, Q3, Q4, Q5: footprint vssop:D2PAK_NEX -> Package_TO_SOT_SMD:TO-263-2
- U1: footprint Package_SO:VSSOP-8_3x3mm_P0.65mm -> Package_SO:VSSOP-10_3x3mm_P0.5mm
Changed lines of the file:
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@@
 			)
 		)
-		(property "Footprint" "vssop:D2PAK_NEX"
+		(property "Footprint" "Package_TO_SOT_SMD:TO-263-2"
 			(at 180.34 19.05 0)
 			(effects
@@
 			)
 		)
-		(property "Footprint" "vssop:D2PAK_NEX"
+		(property "Footprint" "Package_TO_SOT_SMD:TO-263-2"
 			(at 138.43 19.05 0)
 			(effects
@@
 			)
 		)
-		(property "Footprint" "vssop:D2PAK_NEX"
+		(property "Footprint" "Package_TO_SOT_SMD:TO-263-2"
 			(at 158.75 19.05 0)
 			(effects
@@
 			)
 		)
-		(property "Footprint" "vssop:D2PAK_NEX"
+		(property "Footprint" "Package_TO_SOT_SMD:TO-263-2"
 			(at 97.79 19.05 0)
 			(effects
@@
 			)
 		)
-		(property "Footprint" "vssop:D2PAK_NEX"
+		(property "Footprint" "Package_TO_SOT_SMD:TO-263-2"
 			(at 118.11 19.05 0)
 			(effects
@@
 			)
 		)
-		(property "Footprint" "Package_SO:VSSOP-8_3x3mm_P0.65mm"
+		(property "Footprint" "Package_SO:VSSOP-10_3x3mm_P0.5mm"
 			(at 102.108 60.706 90)
 			(effects
@@
 	)
 	(symbol
-		(lib_id "xt90:XT90PW-M")
+		(lib_id "XT90PW-M:XT90PW-M")
 		(at 24.13 25.4 180)
 		(unit 1)

Commit message: fixed ERC
Parts:
- U1: symbol tps2490g:TPS2490DGSR -> TPS2490DGSR:TPS2490DGSR
Changed lines of the file:
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@@
 	)
 	(symbol
-		(lib_id "tps2490g:TPS2490DGSR")
+		(lib_id "TPS2490DGSR:TPS2490DGSR")
 		(at 86.36 59.69 0)
 		(unit 1)
