File: power_switch.kicad_sch (KiCad schematic)
At the start: 19 parts, among them J1 XT90PW-M, Q1 PSMN3R7-100BSEJ, Q2 PSMN3R7-100BSEJ, Q3 PSMN3R7-100BSEJ, Q4 PSMN3R7-100BSEJ, Q5 PSMN3R7-100BSEJ, SW1 SW_SPST, U1 TPS2490

Commit message: moved schematics back to root folder
Parts:
- J1: symbol XT90PW-M:XT90PW-M -> xt90:XT90PW-M
- U1: symbol TPS2490DGSR:TPS2490DGSR -> tps2490g:TPS2490DGSR
Connections:
- net V_switched renamed 48v_switched
Changed lines of the file:
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@@
 		)
 	)
-	(global_label "V_switched"
+	(global_label "48v_switched"
 		(shape input)
 		(at 193.04 13.97 0)
@@
 		)
 		(property "Intersheetrefs" "${INTERSHEET_REFS}"
-			(at 206.2457 13.97 0)
+			(at 208.5437 13.97 0)
 			(effects
 				(font
@@
 	)
 	(symbol
-		(lib_id "TPS2490DGSR:TPS2490DGSR")
+		(lib_id "tps2490g:TPS2490DGSR")
 		(at 86.36 59.69 0)
 		(unit 1)
@@
 	)
 	(symbol
-		(lib_id "XT90PW-M:XT90PW-M")
+		(lib_id "xt90:XT90PW-M")
 		(at 24.13 25.4 180)
 		(unit 1)

Commit message: started routing
Connections:
- net drain: now reaches Q1.MB, Q2.MB, Q3.MB, Q4.MB, Q5.MB, R5.2, U1.9 (SENSE)
Changed lines of the file:
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@@
+		)
+	)
+	(label "drain"
+		(at 101.6 25.4 0)
+		(effects
+			(font
+				(size 1.27 1.27)
+			)
+			(justify left bottom)
 		)
 	)

Commit message: updates
Parts:
- J1: footprint Connector_AMASS:AMASS_XT90PW-M_1x02_P10.90mm_Horizontal -> vssop:AMASS_XT90PW-M
Other:
- moved on the sheet: J1, R5
Changed lines of the file:
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@@
 	)
 	(junction
-		(at 29.21 35.56)
-		(diameter 0)
-		(color 0 0 0 0)
-	)
-	(junction
 		(at 95.25 25.4)
 		(diameter 0)
@@
 	)
 	(junction
-		(at 76.2 35.56)
+		(at 36.83 35.56)
 		(diameter 0)
 		(color 0 0 0 0)
 	)
 	(junction
-		(at 36.83 35.56)
+		(at 60.96 69.85)
 		(diameter 0)
 		(color 0 0 0 0)
 	)
 	(junction
-		(at 60.96 69.85)
+		(at 67.31 35.56)
 		(diameter 0)
 		(color 0 0 0 0)
 	)
 	(junction
-		(at 67.31 35.56)
+		(at 72.39 35.56)
 		(diameter 0)
 		(color 0 0 0 0)
@@
 	)
 	(junction
+		(at 83.82 30.48)
+		(diameter 0)
+		(color 0 0 0 0)
+	)
+	(junction
 		(at 161.29 34.29)
 		(diameter 0)
@@
 	)
 	(junction
-		(at 83.82 33.02)
-		(diameter 0)
-		(color 0 0 0 0)
-	)
-	(junction
 		(at 156.21 13.97)
 		(diameter 0)
@@
 	(wire
 		(pts
-			(xy 67.31 35.56) (xy 76.2 35.56)
+			(xy 67.31 35.56) (xy 72.39 35.56)
 		)
 		(stroke
@@
 	(wire
 		(pts
-			(xy 76.2 35.56) (xy 80.01 35.56)
+			(xy 120.65 34.29) (xy 120.65 16.51)
 		)
 		(stroke
@@
 	(wire
 		(pts
-			(xy 120.65 34.29) (xy 120.65 16.51)
+			(xy 36.83 35.56) (xy 49.53 35.56)
 		)
 		(stroke
@@
 	(wire
 		(pts
-			(xy 36.83 35.56) (xy 49.53 35.56)
+			(xy 80.01 30.48) (xy 83.82 30.48)
 		)
 		(stroke
@@
 	(wire
 		(pts
-			(xy 83.82 33.02) (xy 83.82 43.18)
+			(xy 60.96 71.12) (xy 60.96 69.85)
 		)
 		(stroke
@@
 	(wire
 		(pts
-			(xy 60.96 71.12) (xy 60.96 69.85)
+			(xy 29.21 58.42) (xy 49.53 58.42)
 		)
 		(stroke
@@
 	(wire
 		(pts
-			(xy 29.21 58.42) (xy 49.53 58.42)
+			(xy 97.79 34.29) (xy 100.33 34.29)
 		)
 		(stroke
@@
 	(wire
 		(pts
-			(xy 97.79 34.29) (xy 100.33 34.29)
+			(xy 161.29 34.29) (xy 182.88 34.29)
 		)
 		(stroke
@@
 	(wire
 		(pts
-			(xy 161.29 34.29) (xy 182.88 34.29)
+			(xy 29.21 67.31) (xy 29.21 66.04)
 		)
 		(stroke
@@
 	(wire
 		(pts
-			(xy 29.21 67.31) (xy 29.21 66.04)
+			(xy 72.39 30.48) (xy 72.39 35.56)
 		)
 		(stroke
@@
 	(wire
 		(pts
-			(xy 76.2 33.02) (xy 76.2 35.56)
+			(xy 72.39 35.56) (xy 80.01 35.56)
 		)
 		(stroke
@@
 	(wire
 		(pts
-			(xy 83.82 25.4) (xy 83.82 33.02)
+			(xy 83.82 25.4) (xy 83.82 30.48)
 		)
 		(stroke
@@
 	(wire
 		(pts
-			(xy 29.21 22.86) (xy 29.21 21.59)
+			(xy 25.4 25.4) (xy 25.4 21.59)
 		)
 		(stroke
@@
 	(wire
 		(pts
-			(xy 71.12 62.23) (xy 60.96 62.23)
+			(xy 83.82 30.48) (xy 83.82 43.18)
 		)
 		(stroke
@@
 	(wire
 		(pts
-			(xy 95.25 24.13) (xy 95.25 25.4)
+			(xy 71.12 62.23) (xy 60.96 62.23)
 		)
 		(stroke
@@
 	(wire
 		(pts
-			(xy 100.33 34.29) (xy 100.33 16.51)
+			(xy 95.25 24.13) (xy 95.25 25.4)
 		)
 		(stroke
@@
 	(wire
 		(pts
-			(xy 67.31 36.83) (xy 67.31 35.56)
+			(xy 100.33 34.29) (xy 100.33 16.51)
 		)
 		(stroke
@@
 	(wire
 		(pts
-			(xy 156.21 25.4) (xy 177.8 25.4)
+			(xy 67.31 36.83) (xy 67.31 35.56)
 		)
 		(stroke
@@
 	(wire
 		(pts
-			(xy 29.21 25.4) (xy 29.21 35.56)
+			(xy 156.21 25.4) (xy 177.8 25.4)
 		)
 		(stroke
@@
 	(wire
 		(pts
-			(xy 29.21 21.59) (xy 33.02 21.59)
+			(xy 25.4 21.59) (xy 33.02 21.59)
 		)
 		(stroke
@@
 	(symbol
 		(lib_id "Device:R")
-		(at 80.01 33.02 90)
+		(at 76.2 30.48 90)
 		(unit 1)
 		(exclude_from_sim no)
@@
 		(fields_autoplaced yes)
 		(property "Reference" "R5"
-			(at 80.01 26.67 90)
+			(at 76.2 24.13 90)
 			(effects
 				(font
@@
 		)
 		(property "Value" "0.2mR, 15W"
-			(at 80.01 29.21 90)
+			(at 76.2 26.67 90)
 			(effects
 				(font
@@
 		)
 		(property "Footprint" "Resistor_SMD:R_1206_3216Metric_Pad1.30x1.75mm_HandSolder"
-			(at 80.01 34.798 90)
+			(at 76.2 32.258 90)
 			(effects
 				(font
@@
 		)
 		(property "Datasheet" "~"
-			(at 80.01 33.02 0)
+			(at 76.2 30.48 0)
 			(effects
 				(font
@@
 		)
 		(property "Description" "Resistor"
-			(at 80.01 33.02 0)
+			(at 76.2 30.48 0)
 			(effects
 				(font
@@
 		)
 		(property "Sim.Device" ""
-			(at 80.01 33.02 90)
+			(at 76.2 30.48 90)
 			(effects
 				(font
@@
 		)
 		(property "Sim.Pins" ""
-			(at 80.01 33.02 90)
+			(at 76.2 30.48 90)
 			(effects
 				(font
@@
 		)
 		(property "Sim.Type" ""
-			(at 80.01 33.02 90)
+			(at 76.2 30.48 90)
 			(effects
 				(font
@@
 	)
 	(symbol
+		(lib_id "power:+48V")
+		(at 25.4 27.94 180)
+		(unit 1)
+		(exclude_from_sim no)
+		(in_bom yes)
+		(on_board yes)
+		(dnp no)
+		(fields_autoplaced yes)
+		(property "Reference" "#PWR021"
+			(at 25.4 24.13 0)
+			(effects
+				(font
+					(size 1.27 1.27)
+				)
+				(hide yes)
+			)
+		)
+		(property "Value" "+48V"
+			(at 25.4 33.02 0)
+			(effects
+				(font
+					(size 1.27 1.27)
+				)
+			)
+		)
+		(property "Footprint" ""
+			(at 25.4 27.94 0)
+			(effects
+				(font
+					(size 1.27 1.27)
+				)
+				(hide yes)
+			)
+		)
+		(property "Datasheet" ""
+			(at 25.4 27.94 0)
+			(effects
+				(font
+					(size 1.27 1.27)
+				)
+				(hide yes)
+			)
+		)
+		(property "Description" "Power symbol creates a global label with name \"+48V\""
+			(at 25.4 27.94 0)
+			(effects
+				(font
+					(size 1.27 1.27)
+				)
+				(hide yes)
+			)
+		)
+		(pin "1"
+		)
+		(instances
+			(project "doggie_board"
+				(path "/883cb7fa-3eb5-48d4-9cde-7c11307d94f0/7e8758ce-fdca-4bb6-a847-f546f03772b9"
+					(reference "#PWR021")
+					(unit 1)
+				)
+			)
+		)
+	)
+	(symbol
 		(lib_id "power:GND")
 		(at 29.21 67.31 0)
@@
 	(symbol
 		(lib_id "xt90:XT90PW-M")
-		(at 24.13 25.4 180)
+		(at 20.32 27.94 180)
 		(unit 1)
 		(exclude_from_sim no)
@@
 		(fields_autoplaced yes)
 		(property "Reference" "J1"
-			(at 20.32 15.24 0)
+			(at 16.51 17.78 0)
 			(effects
 				(font
@@
 		)
 		(property "Value" "XT90PW-M"
-			(at 20.32 17.78 0)
+			(at 16.51 20.32 0)
 			(effects
 				(font
@@
 			)
 		)
-		(property "Footprint" "Connector_AMASS:AMASS_XT90PW-M_1x02_P10.90mm_Horizontal"
-			(at 24.13 25.4 0)
+		(property "Footprint" "vssop:AMASS_XT90PW-M"
+			(at 20.32 27.94 0)
 			(effects
 				(font
@@
 		)
 		(property "Datasheet" ""
-			(at 24.13 25.4 0)
+			(at 20.32 27.94 0)
 			(effects
 				(font
@@
 		)
 		(property "Description" ""
-			(at 24.13 25.4 0)
+			(at 20.32 27.94 0)
 			(effects
 				(font
@@
 		)
 		(property "MF" "AMASS"
-			(at 24.13 25.4 0)
+			(at 20.32 27.94 0)
 			(effects
 				(font
@@
 		)
 		(property "Description_1" "Socket; DC supply; XT90; male; PIN: 2; on PCBs; THT; Colour: yellow"
-			(at 24.13 25.4 0)
+			(at 20.32 27.94 0)
 			(effects
 				(font
@@
 		)
 		(property "Package" "Package"
-			(at 24.13 25.4 0)
+			(at 20.32 27.94 0)
 			(effects
 				(font
@@
 		)
 		(property "Price" "None"
-			(at 24.13 25.4 0)
+			(at 20.32 27.94 0)
 			(effects
 				(font
@@
 		)
 		(property "Check_prices" "https://www.snapeda.com/parts/XT90PW-M/AMASS/view-part/?ref=eda"
-			(at 24.13 25.4 0)
+			(at 20.32 27.94 0)
 			(effects
 				(font
@@
 		)
 		(property "MAXIMUM_PACKAGE_HIEGHT" "10.3mm"
-			(at 24.13 25.4 0)
+			(at 20.32 27.94 0)
 			(effects
 				(font
@@
 		)
 		(property "STANDARD" "Manufacturer Recommendations"
-			(at 24.13 25.4 0)
+			(at 20.32 27.94 0)
 			(effects
 				(font
@@
 		)
 		(property "PARTREV" "V00"
-			(at 24.13 25.4 0)
+			(at 20.32 27.94 0)
 			(effects
 				(font
@@
 		)
 		(property "SnapEDA_Link" "https://www.snapeda.com/parts/XT90PW-M/AMASS/view-part/?ref=snap"
-			(at 24.13 25.4 0)
+			(at 20.32 27.94 0)
 			(effects
 				(font
@@
 		)
 		(property "MP" "XT90PW-M"
-			(at 24.13 25.4 0)
+			(at 20.32 27.94 0)
 			(effects
 				(font
@@
 		)
 		(property "Availability" "Not in stock"
-			(at 24.13 25.4 0)
+			(at 20.32 27.94 0)
 			(effects
 				(font
@@
 		)
 		(property "MANUFACTURER" "AMASS"
-			(at 24.13 25.4 0)
+			(at 20.32 27.94 0)
 			(effects
 				(font
@@
 		)
 		(property "Sim.Device" ""
-			(at 24.13 25.4 0)
+			(at 20.32 27.94 0)
 			(effects
 				(font
@@
 		)
 		(property "Sim.Pins" ""
-			(at 24.13 25.4 0)
+			(at 20.32 27.94 0)
 			(effects
 				(font
@@
 		)
 		(property "Sim.Type" ""
-			(at 24.13 25.4 0)
+			(at 20.32 27.94 0)
 			(effects
 				(font

Commit message: progress on routing
Parts:
- D1: value SMF48A -> SMC5K51A-M3/I; footprint Package_SON:WSON-6-1EP_2x2mm_P0.65mm_EP1x1.6mm_ThermalVias -> Diode_SMD:D_SMB-SMC_Universal_Handsoldering
- R5: footprint Resistor_SMD:R_1206_3216Metric_Pad1.30x1.75mm_HandSolder -> vssop:RES_PSR500_ROM
Changed lines of the file:
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@@
 			)
 		)
-		(property "Footprint" "Resistor_SMD:R_1206_3216Metric_Pad1.30x1.75mm_HandSolder"
+		(property "Footprint" "vssop:RES_PSR500_ROM"
 			(at 76.2 32.258 90)
 			(effects
@@
 			)
 		)
-		(property "Value" "SMF48A"
+		(property "Value" "SMC5K51A-M3/I"
 			(at 69.85 41.9099 90)
 			(effects
@@
 			)
 		)
-		(property "Footprint" "Package_SON:WSON-6-1EP_2x2mm_P0.65mm_EP1x1.6mm_ThermalVias"
+		(property "Footprint" "Diode_SMD:D_SMB-SMC_Universal_Handsoldering"
 			(at 62.23 40.64 0)
 			(effects

Commit message: Renaming of Parts
Rename
Parts:
- D1: value SMC5K51A-M3/I -> SMF48A; footprint Diode_SMD:D_SMB-SMC_Universal_Handsoldering -> Package_SON:WSON-6-1EP_2x2mm_P0.65mm_EP1x1.6mm_ThermalVias
- R1: value 212kR -> 212k
- R2: value 10kR -> 10k
- R3: value 100kR -> 100k
- R4: value 18kR -> 18k
- R5: value 0.2mR, 15W -> 0.2m, 15W; footprint vssop:RES_PSR500_ROM -> Resistor_SMD:R_1206_3216Metric_Pad1.30x1.75mm_HandSolder
- R6: value 10R -> 10
- R7: value 1kR -> 1k
Changed lines of the file:
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@@
 			)
 		)
-		(property "Value" "1kR"
+		(property "Value" "1k"
 			(at 187.96 31.75 90)
 			(effects
@@
 			)
 		)
-		(property "Value" "18kR"
+		(property "Value" "18k"
 			(at 63.5 76.1999 0)
 			(effects
@@
 			)
 		)
-		(property "Value" "10kR"
+		(property "Value" "10k"
 			(at 31.75 63.4999 0)
 			(effects
@@
 			)
 		)
-		(property "Value" "0.2mR, 15W"
+		(property "Value" "0.2m, 15W"
 			(at 76.2 26.67 90)
 			(effects
@@
 			)
 		)
-		(property "Footprint" "vssop:RES_PSR500_ROM"
+		(property "Footprint" "Resistor_SMD:R_1206_3216Metric_Pad1.30x1.75mm_HandSolder"
 			(at 76.2 32.258 90)
 			(effects
@@
 			)
 		)
-		(property "Value" "SMC5K51A-M3/I"
+		(property "Value" "SMF48A"
 			(at 69.85 41.9099 90)
 			(effects
@@
 			)
 		)
-		(property "Footprint" "Diode_SMD:D_SMB-SMC_Universal_Handsoldering"
+		(property "Footprint" "Package_SON:WSON-6-1EP_2x2mm_P0.65mm_EP1x1.6mm_ThermalVias"
 			(at 62.23 40.64 0)
 			(effects
@@
 			)
 		)
-		(property "Value" "10R"
+		(property "Value" "10"
 			(at 95.25 31.75 90)
 			(effects
@@
 			)
 		)
-		(property "Value" "100kR"
+		(property "Value" "100k"
 			(at 63.5 67.3099 0)
 			(effects
@@
 			)
 		)
-		(property "Value" "212kR"
+		(property "Value" "212k"
 			(at 31.75 55.8799 0)
 			(effects

Commit message: updated footprints and pcb
Parts:
- R1, R2, R3, R4: footprint Resistor_SMD:R_1206_3216Metric_Pad1.30x1.75mm_HandSolder -> Resistor_SMD:R_0201_0603Metric_Pad0.64x0.40mm_HandSolder
Changed lines of the file:
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@@
 			)
 		)
-		(property "Footprint" "Resistor_SMD:R_1206_3216Metric_Pad1.30x1.75mm_HandSolder"
+		(property "Footprint" "Resistor_SMD:R_0201_0603Metric_Pad0.64x0.40mm_HandSolder"
 			(at 59.182 74.93 90)
 			(effects
@@
 			)
 		)
-		(property "Footprint" "Resistor_SMD:R_1206_3216Metric_Pad1.30x1.75mm_HandSolder"
+		(property "Footprint" "Resistor_SMD:R_0201_0603Metric_Pad0.64x0.40mm_HandSolder"
 			(at 27.432 62.23 90)
 			(effects
@@
 			)
 		)
-		(property "Footprint" "Resistor_SMD:R_1206_3216Metric_Pad1.30x1.75mm_HandSolder"
+		(property "Footprint" "Resistor_SMD:R_0201_0603Metric_Pad0.64x0.40mm_HandSolder"
 			(at 59.182 66.04 90)
 			(effects
@@
 			)
 		)
-		(property "Footprint" "Resistor_SMD:R_1206_3216Metric_Pad1.30x1.75mm_HandSolder"
+		(property "Footprint" "Resistor_SMD:R_0201_0603Metric_Pad0.64x0.40mm_HandSolder"
 			(at 27.432 54.61 90)
 			(effects

Commit message: updates
Parts:
- removed Q4, Q5: PSMN3R7-100BSEJ, Package_TO_SOT_SMD:TO-263-2, symbol PSMN3R7-100BSEJ:PSMN3R7-100BSEJ
- added C1: 0.1uF, 100V, Capacitor_SMD:C_1206_3216Metric_Pad1.33x1.80mm_HandSolder, symbol Device:C_Small
- added C2: 27nF, 100V, Capacitor_SMD:C_1206_3216Metric_Pad1.33x1.80mm_HandSolder, symbol Device:C_Small
- added Ct1: 1nF, Capacitor_SMD:C_0805_2012Metric_Pad1.18x1.45mm_HandSolder, symbol Device:C_Small
- added D1: 15KPA048C-SD-Q, footprints:DIODE_15KPA048C-SD-Q_BRN, symbol Diode:SMF48A
- added J2: XT90PW-M, footprints:AMASS_XT90PW-M, symbol xt90:XT90PW-M
- added Q1, Q2, Q3: PSMN3R7-100BSEJ, Package_TO_SOT_SMD:TO-263-2, symbol PSMN3R7-100BSEJ:PSMN3R7-100BSEJ
- added R15, R16, R17, R7, R8: 50, Resistor_SMD:R_1206_3216Metric_Pad1.30x1.75mm_HandSolder, symbol Device:R_Small
- added R3: 100k, Resistor_SMD:R_0201_0603Metric_Pad0.64x0.40mm_HandSolder, symbol Device:R
- added R4: 18k, Resistor_SMD:R_0201_0603Metric_Pad0.64x0.40mm_HandSolder, symbol Device:R
- added R5: 0.2m, 15W, Resistor_SMD:R_1206_3216Metric_Pad1.30x1.75mm_HandSolder, symbol Device:R
- added R9: 1k, Resistor_SMD:R_1206_3216Metric_Pad1.30x1.75mm_HandSolder, symbol Device:R_Small
- added U1: TPS2490, Package_SO:VSSOP-10_3x3mm_P0.5mm, symbol tps2490g:TPS2490DGSR
- D2: renamed from D1; value SMF48A -> 15KPA048C-SD-Q; footprint Package_SON:WSON-6-1EP_2x2mm_P0.65mm_EP1x1.6mm_ThermalVias -> footprints:DIODE_15KPA048C-SD-Q_BRN
- J1: footprint vssop:AMASS_XT90PW-M -> footprints:AMASS_XT90PW-M
- R6: value 10 -> 50
- renumbered C1 to C3, C2 to C4, Ct1 to Ct2, Q1 to Q4, Q2 to Q5, Q3 to Q6, R3 to R12, R4 to R13, R5 to R14, R7 to R18, U1 to U2
Connections:
- net 48v_switched is gone; now on net +48V: Q4.3, Q5.3, Q6.3, U2.7 (OUT)
- net +48V: now also Q1.3, Q2.3, Q3.3, U1.7 (OUT); no longer C3.1, D2.1 (A1), J1.P (POS), R1.1, R14.1, U2.10 (VCC)
- net GND: now also C1.2, C2.2, Ct1.2, D1.2 (A2), J2.N (NEG), R4.2, U1.5 (GND)
- net drain: now also Q1.MB, Q2.MB, Q3.MB, R5.2, U1.9 (SENSE)
- net gate_line: now also R18.2, R6.1, U2.8 (GATE), R15.1, R16.1, R17.1, R7.1, R8.1, R9.2, U1.8 (GATE); no longer Q4.1, Q5.1, Q6.1, R18.1, R6.2
- net at C4.1: now also R18.1; no longer R18.2
- net ps_sw: now reaches SW1.2 (B), U2.1 (EN)
- net ps_sw: now also U1.1 (EN)
- net SWITCH_HIGH: no longer names the net of R1.2, R2.1, SW1.1 (A)
- new net: Q2.1, R7.2
- new net: Q5.1, R16.2
- new net: R3.1, U1.2 (VREF)
- new net: R3.2, R4.1, U1.3 (PROG)
- new net: Ct1.1, U1.4 (TIMER)
- new net: Q6.1, R17.2
- new net: C2.1, R9.1
- new net: Q3.1, R8.2
- new net: Q4.1, R15.2
- new net: Q1.1, R6.2
- new net 48_L: C1.1, D1.1 (A1), J1.P (POS), R1.1, R5.1, U1.10 (VCC)
- new net 48_R: C3.1, D2.1 (A1), J2.P (POS), R14.1, U2.10 (VCC)
- no-connect marks 1 -> 2
Other:
- moved on the sheet: C3, C4, Ct2, D2, J1, Q4, Q5, Q6, R12, R13, R14, R18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

Commit message: fixed ERC
Connections:
- net drain renamed drain_left
- net drain_left: no longer Q4.MB, Q5.MB, Q6.MB, R14.2, U2.9 (SENSE)
- net gate_line renamed gate_line_left
- net gate_line_left: no longer R15.1, R16.1, R17.1, R18.2, U2.8 (GATE)
- new net drain_r: Q4.MB, Q5.MB, Q6.MB, R14.2, U2.9 (SENSE)
- new net gate_line_r: R15.1, R16.1, R17.1, R18.2, U2.8 (GATE)
Changed lines of the file:
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@@
 		)
 	)
-	(label "drain"
+	(label "drain_r"
 		(at 227.33 41.91 0)
 		(effects
@@
 		)
 	)
-	(label "gate_line"
+	(label "gate_line_r"
 		(at 229.87 50.8 0)
 		(effects
@@
 		)
 	)
-	(label "drain"
-		(at 101.6 41.91 0)
+	(label "drain_left"
+		(at 100.33 41.91 0)
 		(effects
 			(font
@@
 		)
 	)
-	(label "gate_line"
-		(at 104.14 50.8 0)
+	(label "gate_line_left"
+		(at 102.87 50.8 0)
 		(effects
 			(font
