File: doggie_board.kicad_pcb (KiCad board)
At the start: 2 copper layers, 127 x 127.5 mm, 40 parts, among them J1 XT90PW-M, Q1 PSMN3R7-100BSEJ, Q2 PSMN3R7-100BSEJ, Q3 PSMN3R7-100BSEJ, Q4 PSMN3R7-100BSEJ, Q5 PSMN3R7-100BSEJ, U1 TPS2490, U2 LM76005, U3 LM76005

Commit message: updates
Parts:
- added U4: LM76005, Package_DFN_QFN:Texas_RNP0030B_WQFN-30-1EP_4x6mm_P0.5mm_EP1.8x4.5mm, F.Cu at (62.0, 109.3)
- J1: footprint Connector_AMASS:AMASS_XT90PW-M_1x02_P10.90mm_Horizontal -> vssop:AMASS_XT90PW-M
- R5: value 0.2mR, 15W -> 0.2m, 15W; footprint vssop:RES_PSR500_ROM -> Resistor_SMD:R_1206_3216Metric_Pad1.30x1.75mm_HandSolder
- moved Cboot1 65.2 mm to (60.9, 86.6)
- moved Cboot2 65.2 mm to (60.9, 66.5)
- moved Cin1 65.2 mm to (60.9, 89.6)
- moved Cin2 65.2 mm to (60.9, 69.6)
- moved Cinx1 65.2 mm to (60.9, 92.6)
- moved Cinx2 65.2 mm to (60.9, 72.6)
- moved Cout1 65.2 mm to (60.9, 95.6)
- moved Cout2 65.2 mm to (60.9, 75.6)
- moved Coutx1 65.2 mm to (60.9, 98.7)
- moved Coutx2 65.2 mm to (60.9, 78.6)
- moved Cvcc1 65.2 mm to (60.9, 101.7)
- moved Cvcc2 65.2 mm to (60.9, 81.6)
- moved L2 65.2 mm to (67.6, 69.0)
- moved Rfbb1 65.2 mm to (71.2, 93.8)
- moved Rfbb2 65.2 mm to (71.2, 73.8)
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Connections:
- Cin1 pad 1: V_switched -> 48v_switched
- Cin2 pad 1: V_switched -> 48v_switched
- Cinx1 pad 1: V_switched -> 48v_switched
- Cinx2 pad 1: V_switched -> 48v_switched
- Q1 pad 2: (no net) -> /High Side Power Switch/drain
- Q2 pad 2: (no net) -> /High Side Power Switch/drain
- Q3 pad 2: (no net) -> /High Side Power Switch/drain
- Q4 pad 2: (no net) -> /High Side Power Switch/drain
- Q5 pad 2: (no net) -> /High Side Power Switch/drain
- R5 pad 2: Net-(U1-SENSE) -> /High Side Power Switch/drain
- U1 pad 9: Net-(U1-SENSE) -> /High Side Power Switch/drain
- U2 pad 18: V_switched -> 48v_switched
- U2 pad 20: V_switched -> 48v_switched
- U2 pad 21: V_switched -> 48v_switched
- U2 pad 22: V_switched -> 48v_switched
- U3 pad 18: V_switched -> 48v_switched
- U3 pad 20: V_switched -> 48v_switched
- U3 pad 21: V_switched -> 48v_switched
- U3 pad 22: V_switched -> 48v_switched
Routing:
- net (no net): track 73.6 -> 0.00 mm
Other:
- board size 127 x 127.5 mm -> 127 x 127 mm

Commit message: progress on routing
Parts:
- added Cboot3: 470nF, 20mOhm, Capacitor_SMD:C_0805_2012Metric_Pad1.18x1.45mm_HandSolder, F.Cu at (59.0, 67.0)
- added Cinx3: 470nF, 33.996mOhm, Capacitor_SMD:C_0805_2012Metric_Pad1.18x1.45mm_HandSolder, F.Cu at (59.0, 70.0)
- added Cout3: 220uF, 10 mOhm, Capacitor_SMD:C_0805_2012Metric_Pad1.18x1.45mm_HandSolder, F.Cu at (59.0, 73.0)
- added Coutx3: 470nF, 58.782mOhm, Capacitor_SMD:C_0805_2012Metric_Pad1.18x1.45mm_HandSolder, F.Cu at (59.0, 76.0)
- added Cvcc3: 2.2uF, 7.474mOhm, Capacitor_SMD:C_0805_2012Metric_Pad1.18x1.45mm_HandSolder, F.Cu at (59.0, 79.0)
- added J5V1: Conn_01x02, Connector_PinHeader_2.54mm:PinHeader_1x02_P2.54mm_Vertical, F.Cu at (58.9, 58.6)
- added J5V2: Conn_01x02, Connector_PinHeader_2.54mm:PinHeader_1x02_P2.54mm_Vertical, F.Cu at (63.4, 58.6)
- added J5V3: Conn_01x02, Connector_PinHeader_2.54mm:PinHeader_1x02_P2.54mm_Vertical, F.Cu at (68.0, 58.6)
- added J5V4: Conn_01x02, Connector_PinHeader_2.54mm:PinHeader_1x02_P2.54mm_Vertical, F.Cu at (72.6, 58.6)
- added J5V5: Conn_01x02, Connector_PinHeader_2.54mm:PinHeader_1x02_P2.54mm_Vertical, F.Cu at (77.2, 58.6)
- added J5V6: Conn_01x02, Connector_PinHeader_2.54mm:PinHeader_1x02_P2.54mm_Vertical, F.Cu at (81.8, 58.6)
- added J5V7: Conn_01x02, Connector_PinHeader_2.54mm:PinHeader_1x02_P2.54mm_Vertical, F.Cu at (86.4, 58.6)
- added J5V8: Conn_01x02, Connector_PinHeader_2.54mm:PinHeader_1x02_P2.54mm_Vertical, F.Cu at (91.0, 58.6)
- added L1(2)1: 4.7uH, 13.1mOhm, Inductor_SMD:L_6.3x6.3_H3, F.Cu at (65.6, 69.4)
- added Rfbb3: 43.2kOhm, Resistor_SMD:R_0201_0603Metric, F.Cu at (62.6, 74.2)
- added Rfbt3: 100kOhm, Resistor_SMD:R_0201_0603Metric, F.Cu at (62.6, 75.9)
- added Rpgood3: 100kOhm, Resistor_SMD:R_0201_0603Metric, F.Cu at (62.6, 77.7)
- D1: value SMF48A -> SMC5K51A-M3/I; footprint Package_SON:WSON-6-1EP_2x2mm_P0.65mm_EP1x1.6mm_ThermalVias -> Diode_SMD:D_SMB-SMC_Universal_Handsoldering
- R5: value 0.2m, 15W -> 0.2mR, 15W; footprint Resistor_SMD:R_1206_3216Metric_Pad1.30x1.75mm_HandSolder -> vssop:RES_PSR500_ROM
- moved J1 152.0 mm to (137.4, 45.0), turned to 0 degrees
- moved R5 98.5 mm to (116.0, 77.5), turned to 0 degrees
- moved U1 74.8 mm to (110.0, 91.5), turned to 90 degrees
- moved D1 70.7 mm to (110.0, 65.5), turned to 90 degrees
- moved Q1 68.8 mm to (122.8, 91.2), turned to 180 degrees
- moved R1 67.4 mm to (119.5, 68.5), turned to 90 degrees
- moved Q5 52.3 mm to (122.8, 153.0), turned to 180 degrees
- moved C2 51.8 mm to (39.1, 148.0)
- moved Cboot2 51.8 mm to (47.9, 116.7)
- moved Cin1 51.8 mm to (47.9, 139.8)
- moved Cinx1 51.8 mm to (47.9, 142.8)
- moved Cinx2 51.8 mm to (47.9, 122.8)
- moved Cout2 51.8 mm to (47.9, 125.8)
- moved Coutx1 51.8 mm to (47.9, 148.8)
- moved Coutx2 51.8 mm to (47.9, 128.8)
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Connections:
- Q1 pad 2: /High Side Power Switch/drain -> (no net)
- Q2 pad 2: /High Side Power Switch/drain -> (no net)
- Q3 pad 2: /High Side Power Switch/drain -> (no net)
- Q4 pad 2: /High Side Power Switch/drain -> (no net)
- Q5 pad 2: /High Side Power Switch/drain -> (no net)

Commit message: updated footprints and pcb
Parts:
- added J5V10: Conn_01x02, Connector_AMASS:AMASS_XT30PW-F_1x02_P2.50mm_Horizontal, F.Cu at (144.8, 119.5)
- added J5V11: Conn_01x02, Connector_AMASS:AMASS_XT30PW-F_1x02_P2.50mm_Horizontal, F.Cu at (145.3, 104.0)
- added J5V12: Conn_01x02, Connector_AMASS:AMASS_XT30PW-F_1x02_P2.50mm_Horizontal, F.Cu at (145.3, 89.0)
- added J5V13: Conn_01x02, Connector_AMASS:AMASS_XT30PW-F_1x02_P2.50mm_Horizontal, F.Cu at (145.5, 73.5)
- added J5V14: Conn_01x02, Connector_AMASS:AMASS_XT30PW-F_1x02_P2.50mm_Horizontal, F.Cu at (144.8, 151.0)
- added J5V15: Conn_01x02, Connector_AMASS:AMASS_XT30U-F_1x02_P5.0mm_Vertical, F.Cu at (133.5, 133.5)
- added J5V16: Conn_01x02, Connector_AMASS:AMASS_XT30U-F_1x02_P5.0mm_Vertical, F.Cu at (134.5, 118.0)
- added J5V17: Conn_01x02, Connector_AMASS:AMASS_XT30U-F_1x02_P5.0mm_Vertical, F.Cu at (133.0, 151.0)
- added J5V18: Conn_01x02, Connector_AMASS:AMASS_XT30U-F_1x02_P5.0mm_Vertical, F.Cu at (135.0, 102.5)
- added J5V19: Conn_01x02, Connector_AMASS:AMASS_XT30U-F_1x02_P5.0mm_Vertical, F.Cu at (135.0, 73.0)
- added J5V20: Conn_01x02, Connector_AMASS:AMASS_XT30U-F_1x02_P5.0mm_Vertical, F.Cu at (136.5, 87.5)
- added J5V9: Conn_01x02, Connector_AMASS:AMASS_XT30PW-F_1x02_P2.50mm_Horizontal, F.Cu at (144.8, 135.5)
- D1: value SMC5K51A-M3/I -> SMF48A; footprint Diode_SMD:D_SMB-SMC_Universal_Handsoldering -> Package_SON:WSON-6-1EP_2x2mm_P0.65mm_EP1x1.6mm_ThermalVias
- R1: value 212kR -> 212k; footprint Resistor_SMD:R_1206_3216Metric_Pad1.30x1.75mm_HandSolder -> Resistor_SMD:R_0201_0603Metric_Pad0.64x0.40mm_HandSolder
- R2: value 10kR -> 10k; footprint Resistor_SMD:R_1206_3216Metric_Pad1.30x1.75mm_HandSolder -> Resistor_SMD:R_0201_0603Metric_Pad0.64x0.40mm_HandSolder
- R3: value 100kR -> 100k; footprint Resistor_SMD:R_1206_3216Metric_Pad1.30x1.75mm_HandSolder -> Resistor_SMD:R_0201_0603Metric_Pad0.64x0.40mm_HandSolder
- R4: value 18kR -> 18k; footprint Resistor_SMD:R_1206_3216Metric_Pad1.30x1.75mm_HandSolder -> Resistor_SMD:R_0201_0603Metric_Pad0.64x0.40mm_HandSolder
- R5: value 0.2mR, 15W -> 0.2m, 15W; footprint vssop:RES_PSR500_ROM -> Resistor_SMD:R_1206_3216Metric_Pad1.30x1.75mm_HandSolder
- R6: value 10R -> 10
- R7: value 1kR -> 1k
- Rfbb1: value 9.09kOhm -> 9.09k
- Rfbb3: value 43.2kOhm -> 43.2k
- Rfbt1, Rfbt2, Rfbt3, Rpgood1, Rpgood2, Rpgood3: value 100kOhm -> 100k
- moved J5V8 68.3 mm to (33.5, 95.5)
- moved J5V6 52.0 mm to (49.0, 99.0)
- moved J5V1 21.1 mm to (41.5, 70.7)
- moved R5 20.4 mm to (119.5, 57.5), turned to -90 degrees
- moved U1 17.9 mm to (95.5, 81.0)
- moved Q1 15.4 mm to (107.5, 93.0)
- moved Q2 14.4 mm to (108.6, 108.8)
- moved Q3 14.4 mm to (108.6, 124.3)
- moved Q4 14.4 mm to (108.7, 139.6)
- moved Q5 14.4 mm to (108.7, 155.1)
- moved R1 7.82 mm to (123.1, 61.5), turned to 180 degrees
Other:
- board size 127 x 127 mm -> 128 x 129 mm

Commit message: updates
Parts:
- added C3: 0.1uF, 100V, Capacitor_SMD:C_1206_3216Metric_Pad1.33x1.80mm_HandSolder, F.Cu at (79.0, 98.9)
- added C4: 27nF, 100V, Capacitor_SMD:C_1206_3216Metric_Pad1.33x1.80mm_HandSolder, F.Cu at (79.0, 102.2)
- added Ct2: 1nF, Capacitor_SMD:C_0805_2012Metric_Pad1.18x1.45mm_HandSolder, F.Cu at (84.4, 98.7)
- added D2: 15KPA048C-SD-Q, footprints:DIODE_15KPA048C-SD-Q_BRN, F.Cu at (63.8, 95.7)
- added J2: XT90PW-M, Connector_AMASS:AMASS_XT90PW-M_1x02_P10.90mm_Horizontal, F.Cu at (63.5, 51.0)
- added Q6: PSMN3R7-100BSEJ, Package_TO_SOT_SMD:TO-263-2, F.Cu at (80.8, 91.0)
- added R10: 50, Resistor_SMD:R_1206_3216Metric_Pad1.30x1.75mm_HandSolder, F.Cu at (80.5, 113.4)
- added R11: 50, Resistor_SMD:R_1206_3216Metric_Pad1.30x1.75mm_HandSolder, F.Cu at (80.5, 116.7)
- added R12: 100k, Resistor_SMD:R_0201_0603Metric_Pad0.64x0.40mm_HandSolder, F.Cu at (80.5, 120.0)
- added R13: 18k, Resistor_SMD:R_0201_0603Metric_Pad0.64x0.40mm_HandSolder, F.Cu at (83.4, 101.1)
- added R14: 0.2m, 15W, Resistor_SMD:R_1206_3216Metric_Pad1.30x1.75mm_HandSolder, F.Cu at (73.0, 98.9)
- added R15: 50, Resistor_SMD:R_1206_3216Metric_Pad1.30x1.75mm_HandSolder, F.Cu at (73.0, 102.2)
- added R16: 50, Resistor_SMD:R_1206_3216Metric_Pad1.30x1.75mm_HandSolder, F.Cu at (73.0, 105.5)
- added R17: 50, Resistor_SMD:R_1206_3216Metric_Pad1.30x1.75mm_HandSolder, F.Cu at (73.0, 108.8)
- added R18: 1k, Resistor_SMD:R_1206_3216Metric_Pad1.30x1.75mm_HandSolder, F.Cu at (73.0, 112.1)
- added R8: 50, Resistor_SMD:R_1206_3216Metric_Pad1.30x1.75mm_HandSolder, F.Cu at (80.5, 106.8)
- added R9: 1k, Resistor_SMD:R_1206_3216Metric_Pad1.30x1.75mm_HandSolder, F.Cu at (80.5, 110.1)
- added U5: LM76005, Package_DFN_QFN:Texas_RNP0030B_WQFN-30-1EP_4x6mm_P0.5mm_EP1.8x4.5mm, F.Cu at (93.3, 89.0)
- D1: value SMF48A -> 15KPA048C-SD-Q; footprint Package_SON:WSON-6-1EP_2x2mm_P0.65mm_EP1x1.6mm_ThermalVias -> footprints:DIODE_15KPA048C-SD-Q_BRN
- J1: footprint vssop:AMASS_XT90PW-M -> Connector_AMASS:AMASS_XT90PW-M_1x02_P10.90mm_Horizontal
- J5V1, J5V2, J5V3, J5V4, J5V5, J5V6, J5V7, J5V8: footprint Connector_PinHeader_2.54mm:PinHeader_1x02_P2.54mm_Vertical -> Connector_AMASS:AMASS_XT30U-F_1x02_P5.0mm_Vertical
- J5V10, J5V11, J5V12, J5V9: footprint Connector_AMASS:AMASS_XT30PW-F_1x02_P2.50mm_Horizontal -> Connector_AMASS:AMASS_XT30U-F_1x02_P5.0mm_Vertical
- J5V13, J5V14: footprint Connector_AMASS:AMASS_XT30PW-F_1x02_P2.50mm_Horizontal -> Connector_PinHeader_2.54mm:PinHeader_1x02_P2.54mm_Vertical
- J5V15, J5V16, J5V17, J5V18, J5V19, J5V20: footprint Connector_AMASS:AMASS_XT30U-F_1x02_P5.0mm_Vertical -> Connector_PinHeader_2.54mm:PinHeader_1x02_P2.54mm_Vertical
- R6: value 10 -> 50
- R7: value 1k -> 50
- U2: value LM76005 -> TPS2490; footprint Package_DFN_QFN:Texas_RNP0030B_WQFN-30-1EP_4x6mm_P0.5mm_EP1.8x4.5mm_ThermalVias -> Package_SO:VSSOP-10_3x3mm_P0.5mm
- U3: footprint Package_DFN_QFN:Texas_RNP0030B_WQFN-30-1EP_4x6mm_P0.5mm_EP1.8x4.5mm -> Package_DFN_QFN:Texas_RNP0030B_WQFN-30-1EP_4x6mm_P0.5mm_EP1.8x4.5mm_ThermalVias
- moved D1 24.6 mm to (134.2, 61.0), turned to -90 degrees
- moved R1 21.6 mm to (104.5, 50.5)
- moved Q1 19.2 mm to (118.1, 77.0)
- moved Q2 18.6 mm to (118.1, 92.8)
- moved Q3 16.9 mm to (118.1, 110.3)
- moved Q4 15.3 mm to (118.0, 127.5)
- moved Q5 13.9 mm to (117.4, 144.3)
- moved J1 6.76 mm to (144.2, 44.7), turned to -90 degrees
- moved J5V20 1.80 mm to (135.0, 88.5)
Connections:
- net /High Side Power Switch/SWITCH_HIGH renamed Net-(SW1-A)
- C1 pad 1: +48V -> 48_L
- Cboot1 pad 1: Net-(U2-BOOT) -> Net-(U3-BOOT)
- Cboot2 pad 1: Net-(U3-BOOT) -> Net-(U4-BOOT)
- Cboot3 pad 1: Net-(U4-BOOT) -> Net-(U5-BOOT)
- Cvcc1 pad 1: Net-(U2-VCC) -> Net-(U3-VCC)
- Cvcc2 pad 1: Net-(U3-VCC) -> Net-(U4-VCC)
- Cvcc3 pad 1: Net-(U4-VCC) -> Net-(U5-VCC)
- D1 pad 1: +48V -> 48_L
- J5V1 pad 1: +5V -> 48v_switched
- J5V10 pad 1: +48V -> 48v_switched
- J5V11 pad 1: +48V -> 48v_switched
- J5V12 pad 1: +48V -> 48v_switched
- J5V13 pad 1: +48V -> +3.3V
- J5V14 pad 1: +48V -> +3.3V
- J5V15 pad 1: +48V -> +3.3V
- J5V16 pad 1: +48V -> +3.3V
- J5V17 pad 1: +48V -> +5V
- J5V18 pad 1: +48V -> +5V
- J5V19 pad 1: +48V -> +5V
- J5V2 pad 1: +5V -> 48v_switched
- J5V20 pad 1: +48V -> +5V
- J5V3 pad 1: +5V -> 48v_switched
- J5V4 pad 1: +5V -> 48v_switched
- J5V5 pad 1: +3.3V -> 48v_switched
- J5V6 pad 1: +3.3V -> 48v_switched
- J5V7 pad 1: +3.3V -> 48v_switched
- J5V8 pad 1: +3.3V -> 48v_switched
- J5V9 pad 1: +48V -> 48v_switched
- Q1 pad 1: /High Side Power Switch/gate_line -> Net-(Q1-Pad1)
- Q1 pad 3: 48v_switched -> +48V
- Q2 pad 1: /High Side Power Switch/gate_line -> Net-(Q2-Pad1)
- Q2 pad 3: 48v_switched -> +48V
- Q3 pad 1: /High Side Power Switch/gate_line -> Net-(Q3-Pad1)
- Q3 pad 3: 48v_switched -> +48V
- Q4 pad 1: /High Side Power Switch/gate_line -> Net-(Q4-Pad1)
- Q4 pad 3: 48v_switched -> +48V
- Q5 pad 1: /High Side Power Switch/gate_line -> Net-(Q5-Pad1)
- Q5 pad 3: 48v_switched -> +48V
- R1 pad 1: +48V -> 48_L
- R5 pad 1: +48V -> 48_L
- R6 pad 1: Net-(U1-GATE) -> /High Side Power Switch/gate_line
- R6 pad 2: /High Side Power Switch/gate_line -> Net-(Q1-Pad1)
- R7 pad 2: Net-(C2-Pad1) -> Net-(Q2-Pad1)
- Rfbb1 pad 1: Net-(U2-FB) -> Net-(U3-FB)
- Rfbb2 pad 1: Net-(U3-FB) -> Net-(U4-FB)
- Rfbb3 pad 1: Net-(U4-FB) -> Net-(U5-FB)
- Rfbt1 pad 2: Net-(U2-FB) -> Net-(U3-FB)
- Rfbt2 pad 2: Net-(U3-FB) -> Net-(U4-FB)
- Rfbt3 pad 2: Net-(U4-FB) -> Net-(U5-FB)
- Rpgood1 pad 1: Net-(U2-PGOOD) -> Net-(U3-PGOOD)
- Rpgood2 pad 1: Net-(U3-PGOOD) -> Net-(U4-PGOOD)
- Rpgood3 pad 2: Net-(U4-PGOOD) -> Net-(U5-PGOOD)
- U1 pad 1: Net-(SW1-B) -> ps_sw
- U1 pad 10: +48V -> 48_L
- U1 pad 7: 48v_switched -> +48V
- U1 pad 8: Net-(U1-GATE) -> /High Side Power Switch/gate_line
- U2 pad 1: Net-(Cboot1-Pad2) -> ps_sw
- U2 pad 10: unconnected-(U2-RT-Pad10) -> 48_R
- U2 pad 2: Net-(Cboot1-Pad2) -> Net-(U2-VREF)
- U2 pad 3: Net-(Cboot1-Pad2) -> Net-(U2-PROG)
- U2 pad 4: Net-(Cboot1-Pad2) -> Net-(U2-TIMER)
- U2 pad 5: Net-(Cboot1-Pad2) -> GND
- U2 pad 6: Net-(U2-BOOT) -> unconnected-(U2-PG-Pad6)
- U2 pad 7: unconnected-(U2-NC-Pad7) -> +48V
- U2 pad 8: Net-(U2-VCC) -> /High Side Power Switch/gate_line
- U2 pad 9: GND -> /High Side Power Switch/drain
- U3 pad 1: Net-(Cboot2-Pad2) -> Net-(Cboot1-Pad2)
- U3 pad 10: GND -> unconnected-(U3-RT-Pad10)
- U3 pad 11: GND -> unconnected-(U3-SS/TRK-Pad11)
- U3 pad 2: Net-(Cboot2-Pad2) -> Net-(Cboot1-Pad2)
- U3 pad 3: Net-(Cboot2-Pad2) -> Net-(Cboot1-Pad2)
- U3 pad 4: Net-(Cboot2-Pad2) -> Net-(Cboot1-Pad2)
- U3 pad 5: Net-(Cboot2-Pad2) -> Net-(Cboot1-Pad2)
- U4 pad 1: Net-(Cboot3-Pad2) -> Net-(Cboot2-Pad2)
- U4 pad 10: unconnected-(U4-RT-Pad10) -> GND
- U4 pad 11: unconnected-(U4-SS/TRK-Pad11) -> GND
- U4 pad 2: Net-(Cboot3-Pad2) -> Net-(Cboot2-Pad2)
- U4 pad 3: Net-(Cboot3-Pad2) -> Net-(Cboot2-Pad2)
- U4 pad 4: Net-(Cboot3-Pad2) -> Net-(Cboot2-Pad2)
- U4 pad 5: Net-(Cboot3-Pad2) -> Net-(Cboot2-Pad2)
Other:
- board size 128 x 129 mm -> 127 x 127.5 mm

Commit message: imported schematic
Parts:
- J1, J2: footprint Connector_AMASS:AMASS_XT90PW-M_1x02_P10.90mm_Horizontal -> footprints:AMASS_XT90PW-M
- moved D1 17.1 mm to (124.3, 47.0)

Commit message: fixed ERC
Parts:
- J5V1, J5V10, J5V11, J5V12, J5V2, J5V3, J5V4, J5V5, J5V6, J5V7, J5V8, J5V9: footprint Connector_AMASS:AMASS_XT30U-F_1x02_P5.0mm_Vertical -> Connector_AMASS:AMASS_XT30PW-M_1x02_P2.50mm_Horizontal
- moved J5V15 104.4 mm to (228.0, 89.1), turned to 0 degrees
- moved U2 101.6 mm to (108.2, 61.5)
- moved J5V17 84.1 mm to (204.4, 106.5)
- moved J5V16 83.5 mm to (212.5, 88.1), turned to 0 degrees
- moved J5V14 74.3 mm to (211.7, 118.5)
- moved J5V18 63.8 mm to (197.0, 87.6), turned to 0 degrees
- moved D1 15.9 mm to (130.4, 61.7)
- turned J1 to 90 degrees
Connections:
- R14 pad 2: /High Side Power Switch/drain -> /High Side Power Switch/drain_r
- R15 pad 1: /High Side Power Switch/gate_line -> /High Side Power Switch/gate_line_r
- R16 pad 1: /High Side Power Switch/gate_line -> /High Side Power Switch/gate_line_r
- R17 pad 1: /High Side Power Switch/gate_line -> /High Side Power Switch/gate_line_r
- R18 pad 2: /High Side Power Switch/gate_line -> /High Side Power Switch/gate_line_r
- R5 pad 2: /High Side Power Switch/drain -> /High Side Power Switch/drain_left
- R6 pad 1: /High Side Power Switch/gate_line -> /High Side Power Switch/gate_line_left
- R7 pad 1: /High Side Power Switch/gate_line -> /High Side Power Switch/gate_line_left
- R8 pad 1: /High Side Power Switch/gate_line -> /High Side Power Switch/gate_line_left
- R9 pad 2: /High Side Power Switch/gate_line -> /High Side Power Switch/gate_line_left
- U1 pad 8: /High Side Power Switch/gate_line -> /High Side Power Switch/gate_line_left
- U1 pad 9: /High Side Power Switch/drain -> /High Side Power Switch/drain_left
- U2 pad 8: /High Side Power Switch/gate_line -> /High Side Power Switch/gate_line_r
- U2 pad 9: /High Side Power Switch/drain -> /High Side Power Switch/drain_r

Commit message: routing progress
Parts:
- removed R17: 50, Resistor_SMD:R_1206_3216Metric_Pad1.30x1.75mm_HandSolder
- removed R18: 1k, Resistor_SMD:R_1206_3216Metric_Pad1.30x1.75mm_HandSolder
- J5V13, J5V14, J5V15, J5V16, J5V17, J5V18, J5V19, J5V20: footprint Connector_PinHeader_2.54mm:PinHeader_1x02_P2.54mm_Vertical -> Connector_PinHeader_1.00mm:PinHeader_1x02_P1.00mm_Vertical
- R10: value 50 -> 100k; footprint Resistor_SMD:R_1206_3216Metric_Pad1.30x1.75mm_HandSolder -> Resistor_SMD:R_0201_0603Metric_Pad0.64x0.40mm_HandSolder
- R11: value 50 -> 18k; footprint Resistor_SMD:R_1206_3216Metric_Pad1.30x1.75mm_HandSolder -> Resistor_SMD:R_0201_0603Metric_Pad0.64x0.40mm_HandSolder
- R12: value 100k -> 0.2m, 15W; footprint Resistor_SMD:R_0201_0603Metric_Pad0.64x0.40mm_HandSolder -> footprints:RES_PSR500_ROM
- R13: value 18k -> 50; footprint Resistor_SMD:R_0201_0603Metric_Pad0.64x0.40mm_HandSolder -> Resistor_SMD:R_1206_3216Metric_Pad1.30x1.75mm_HandSolder
- R14: value 0.2m, 15W -> 50
- R16: value 50 -> 1k
- R5: footprint Resistor_SMD:R_1206_3216Metric_Pad1.30x1.75mm_HandSolder -> footprints:RES_PSR500_ROM
- moved R6 193.8 mm to (222.1, 69.5)
- moved R2 137.8 mm to (186.2, 49.9)
- moved Cboot1 127.2 mm to (169.3, 174.6)
- moved Cout1 127.2 mm to (169.3, 183.6)
- moved Cboot2 127.2 mm to (169.3, 154.5)
- moved Cin1 127.2 mm to (169.3, 177.6)
- moved Cin2 127.2 mm to (169.3, 157.5)
- moved Cinx1 127.2 mm to (169.3, 180.6)
- moved Cinx2 127.2 mm to (169.3, 160.5)
- moved Cout2 127.2 mm to (169.3, 163.5)
- moved Coutx1 127.2 mm to (169.3, 186.6)
- moved Coutx2 127.2 mm to (169.3, 166.5)
- moved Cvcc1 127.2 mm to (169.3, 189.6)
- moved Cvcc2 127.2 mm to (169.3, 169.5)
- moved U3 127.2 mm to (175.3, 165.0)
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Connections:
- Cin1 pad 1: 48v_switched -> +48V
- Cin2 pad 1: 48v_switched -> +48V
- Cinx1 pad 1: 48v_switched -> +48V
- Cinx2 pad 1: 48v_switched -> +48V
- Cinx3 pad 1: 48v_switched -> +48V
- J5V1 pad 1: 48v_switched -> +48V
- J5V10 pad 1: 48v_switched -> +48V
- J5V11 pad 1: 48v_switched -> +48V
- J5V12 pad 1: 48v_switched -> +48V
- J5V2 pad 1: 48v_switched -> +48V
- J5V3 pad 1: 48v_switched -> +48V
- J5V4 pad 1: 48v_switched -> +48V
- J5V5 pad 1: 48v_switched -> +48V
- J5V6 pad 1: 48v_switched -> +48V
- J5V7 pad 1: 48v_switched -> +48V
- J5V8 pad 1: 48v_switched -> +48V
- J5V9 pad 1: 48v_switched -> +48V
- R10 pad 1: /High Side Power Switch/gate_line -> Net-(U2-VREF)
- R10 pad 2: Net-(Q3-Pad1) -> Net-(U2-PROG)
- R11 pad 1: /High Side Power Switch/gate_line -> Net-(U2-PROG)
- R11 pad 2: Net-(Q4-Pad1) -> GND
- R12 pad 1: Net-(U2-VREF) -> 48_R
- R12 pad 2: Net-(U2-PROG) -> /High Side Power Switch/drain_r
- R13 pad 1: Net-(U2-PROG) -> /High Side Power Switch/gate_line_r
- R13 pad 2: GND -> Net-(Q4-Pad1)
- R14 pad 1: 48_R -> /High Side Power Switch/gate_line_r
- R14 pad 2: /High Side Power Switch/drain_r -> Net-(Q5-Pad1)
- R15 pad 2: Net-(Q4-Pad1) -> Net-(Q6-Pad1)
- R16 pad 1: /High Side Power Switch/gate_line_r -> Net-(C4-Pad1)
- R16 pad 2: Net-(Q5-Pad1) -> /High Side Power Switch/gate_line_r
- U3 pad 18: 48v_switched -> +48V
- U3 pad 20: 48v_switched -> +48V
- U3 pad 21: 48v_switched -> +48V
- U3 pad 22: 48v_switched -> +48V
- U4 pad 18: 48v_switched -> +48V
- U4 pad 20: 48v_switched -> +48V
- U4 pad 21: 48v_switched -> +48V
- U4 pad 22: 48v_switched -> +48V
- U5 pad 18: 48v_switched -> +48V
- U5 pad 20: 48v_switched -> +48V
- U5 pad 21: 48v_switched -> +48V
- U5 pad 22: 48v_switched -> +48V
Routing:
- added copper zone on F.Cu, net +48V

Commit message: transistor pins
Routing:
- net (no net): vias 0 -> 1
Changed lines of the file:
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@@
 		(layer "Edge.Cuts")
+	)
+	(via
+		(at 131.4 126.45)
+		(size 1)
+		(drill 0.8)
+		(layers "F.Cu" "B.Cu")
+		(free yes)
+		(net 0)
 	)
 	(zone
