File: buck5v.kicad_sch (KiCad schematic)
At the start: 15 parts, among them U3 TPS566242DRLR

Commit message: feat: added footprints
Parts:
- C10, C11, C12, C13, C14, C15, C16, C17, C18, L2: footprint (none) -> Capacitor_SMD:C_0201_0603Metric_Pad0.64x0.40mm_HandSolder
- R19, R20, R21, R22: footprint (none) -> Resistor_SMD:R_0201_0603Metric_Pad0.64x0.40mm_HandSolder
Changed lines of the file:
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@@
 			)
 		)
-		(property "Footprint" ""
+		(property "Footprint" "Capacitor_SMD:C_0201_0603Metric_Pad0.64x0.40mm_HandSolder"
 			(at 120.65 34.29 0)
 			(effects
@@
 			)
 		)
-		(property "Footprint" ""
+		(property "Footprint" "Resistor_SMD:R_0201_0603Metric_Pad0.64x0.40mm_HandSolder"
 			(at 43.18 44.45 0)
 			(effects
@@
 			)
 		)
-		(property "Footprint" ""
+		(property "Footprint" "Capacitor_SMD:C_0201_0603Metric_Pad0.64x0.40mm_HandSolder"
 			(at 99.06 31.75 0)
 			(effects
@@
 			)
 		)
-		(property "Footprint" ""
+		(property "Footprint" "Capacitor_SMD:C_0201_0603Metric_Pad0.64x0.40mm_HandSolder"
 			(at 137.16 34.29 0)
 			(effects
@@
 			)
 		)
-		(property "Footprint" ""
+		(property "Footprint" "Capacitor_SMD:C_0201_0603Metric_Pad0.64x0.40mm_HandSolder"
 			(at 154.94 34.29 0)
 			(effects
@@
 			)
 		)
-		(property "Footprint" ""
+		(property "Footprint" "Resistor_SMD:R_0201_0603Metric_Pad0.64x0.40mm_HandSolder"
 			(at 43.18 36.83 0)
 			(effects
@@
 			)
 		)
-		(property "Footprint" ""
+		(property "Footprint" "Capacitor_SMD:C_0201_0603Metric_Pad0.64x0.40mm_HandSolder"
 			(at 146.05 34.29 0)
 			(effects
@@
 			)
 		)
-		(property "Footprint" ""
+		(property "Footprint" "Capacitor_SMD:C_0201_0603Metric_Pad0.64x0.40mm_HandSolder"
 			(at 16.51 36.83 0)
 			(effects
@@
 			)
 		)
-		(property "Footprint" ""
+		(property "Footprint" "Resistor_SMD:R_0201_0603Metric_Pad0.64x0.40mm_HandSolder"
 			(at 110.49 41.91 0)
 			(effects
@@
 			)
 		)
-		(property "Footprint" ""
+		(property "Footprint" "Capacitor_SMD:C_0201_0603Metric_Pad0.64x0.40mm_HandSolder"
 			(at 25.4 36.83 0)
 			(effects
@@
 			)
 		)
-		(property "Footprint" ""
+		(property "Footprint" "Capacitor_SMD:C_0201_0603Metric_Pad0.64x0.40mm_HandSolder"
 			(at 34.29 36.83 0)
 			(effects
@@
 			)
 		)
-		(property "Footprint" ""
+		(property "Footprint" "Capacitor_SMD:C_0201_0603Metric_Pad0.64x0.40mm_HandSolder"
 			(at 102.87 34.29 0)
 			(effects
@@
 			)
 		)
-		(property "Footprint" ""
+		(property "Footprint" "Capacitor_SMD:C_0201_0603Metric_Pad0.64x0.40mm_HandSolder"
 			(at 128.27 34.29 0)
 			(effects
@@
 			)
 		)
-		(property "Footprint" ""
+		(property "Footprint" "Resistor_SMD:R_0201_0603Metric_Pad0.64x0.40mm_HandSolder"
 			(at 110.49 34.29 0)
 			(effects

Commit message: added headers and modified some stuff
Parts:
- added J7: Conn_01x03, symbol Connector_Generic:Conn_01x03
- added Q11: 2N7002, Package_TO_SOT_SMD:SOT-23, symbol Transistor_FET:2N7002
Connections:
- net GND: now also J7.3 (Pin_3)
- net EN renamed +5V_EN
- net +5V_EN: now also J7.1 (Pin_1); no longer U3.5 (EN)
- new net: Q11.2 (S), U3.5 (EN)
- new net 12V_PG: Q11.1 (G)
- new net 5V_EN: J7.2 (Pin_2), Q11.3 (D)
Other:
- note added: "Bridge 1 and 2 for always on NMOS adds sequensing (wait for 12V rail good)"
- moved on the sheet: R19, R20

Commit message: added footprints and standardized EN headers
Parts:
- J7: footprint (none) -> Connector_PinHeader_2.54mm:PinHeader_1x03_P2.54mm_Vertical
Connections:
- net +5V_EN renamed +5V_LP
Changed lines of the file:
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@@
+	(wire
+		(pts
+			(xy 133.35 49.53) (xy 135.89 49.53)
+		)
+		(stroke
+			(width 0)
+			(type default)
+		)
+	)
 	(wire
 		(pts
@@
 	(wire
 		(pts
+			(xy 99.06 55.88) (xy 99.06 54.61)
+		)
+		(stroke
+			(width 0)
+			(type default)
+		)
+	)
+	(wire
+		(pts
 			(xy 110.49 31.75) (xy 120.65 31.75)
 		)
@@
 			(width 0)
 			(type default)
+		)
+	)
+	(label "5V_EN"
+		(at 99.06 55.88 0)
+		(effects
+			(font
+				(size 1.27 1.27)
+			)
+			(justify left bottom)
 		)
 	)
@@
 		)
 	)
-	(global_label "5V_EN"
-		(shape input)
-		(at 99.06 54.61 0)
-		(fields_autoplaced yes)
+	(label "5V_EN"
+		(at 133.35 49.53 180)
 		(effects
 			(font
 				(size 1.27 1.27)
 			)
-			(justify left)
-		)
-		(property "Intersheetrefs" "${INTERSHEET_REFS}"
-			(at 107.7904 54.61 0)
-			(effects
-				(font
-					(size 1.27 1.27)
-				)
-				(justify left)
-				(hide yes)
-			)
+			(justify right bottom)
 		)
 	)
@@
 		)
 	)
-	(global_label "5V_EN"
-		(shape input)
-		(at 135.89 49.53 180)
-		(fields_autoplaced yes)
-		(effects
-			(font
-				(size 1.27 1.27)
-			)
-			(justify right)
-		)
-		(property "Intersheetrefs" "${INTERSHEET_REFS}"
-			(at 127.1596 49.53 0)
-			(effects
-				(font
-					(size 1.27 1.27)
-				)
-				(justify right)
-				(hide yes)
-			)
-		)
-	)
 	(symbol
 		(lib_id "Device:C_Small")
@@
 			)
 		)
-		(property "Value" "+5V_EN"
-			(at 132.08 46.9899 90)
-			(effects
-				(font
-					(size 1.27 1.27)
-				)
-				(justify left)
+		(property "Value" "+5V_LP"
+			(at 134.62 44.45 90)
+			(effects
+				(font
+					(size 1.27 1.27)
+				)
 			)
 		)
@@
 			)
 		)
-		(property "Value" "+5V_EN"
+		(property "Value" "+5V_LP"
 			(at 26.67 66.0399 90)
 			(effects
@@
 			)
 		)
-		(property "Footprint" ""
+		(property "Footprint" "Connector_PinHeader_2.54mm:PinHeader_1x03_P2.54mm_Vertical"
 			(at 140.97 49.53 0)
 			(effects

Commit message: final push
Parts:
- L2: footprint Capacitor_SMD:C_0201_0603Metric_Pad0.64x0.40mm_HandSolder -> footprints:IND_1217AS-H-2R2N=P3
Changed lines of the file:
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@@
 		)
 		(instances
+			(project "buck5v"
+				(path "/45bff242-0d9b-4726-901e-ccb01efc2321"
+					(reference "C?")
+					(unit 1)
+				)
+			)
 			(project "doggie_board"
 				(path "/883cb7fa-3eb5-48d4-9cde-7c11307d94f0/64e74d8d-15e7-49a6-a99b-9f52cddf6628"
@@
 		)
 		(instances
+			(project "buck5v"
+				(path "/45bff242-0d9b-4726-901e-ccb01efc2321"
+					(reference "R?")
+					(unit 1)
+				)
+			)
 			(project "doggie_board"
 				(path "/883cb7fa-3eb5-48d4-9cde-7c11307d94f0/64e74d8d-15e7-49a6-a99b-9f52cddf6628"
@@
 		)
 		(instances
+			(project "buck5v"
+				(path "/45bff242-0d9b-4726-901e-ccb01efc2321"
+					(reference "#PWR?")
+					(unit 1)
+				)
+			)
 			(project "doggie_board"
 				(path "/883cb7fa-3eb5-48d4-9cde-7c11307d94f0/64e74d8d-15e7-49a6-a99b-9f52cddf6628"
@@
 			)
 		)
-		(property "Footprint" "Capacitor_SMD:C_0201_0603Metric_Pad0.64x0.40mm_HandSolder"
+		(property "Footprint" "footprints:IND_1217AS-H-2R2N=P3"
 			(at 99.06 31.75 0)
 			(effects
@@
 		)
 		(instances
+			(project "buck5v"
+				(path "/45bff242-0d9b-4726-901e-ccb01efc2321"
+					(reference "L?")
+					(unit 1)
+				)
+			)
 			(project ""
 				(path "/883cb7fa-3eb5-48d4-9cde-7c11307d94f0/64e74d8d-15e7-49a6-a99b-9f52cddf6628"
@@
 		)
 		(instances
+			(project "buck5v"
+				(path "/45bff242-0d9b-4726-901e-ccb01efc2321"
+					(reference "Q?")
+					(unit 1)
+				)
+			)
 			(project ""
 				(path "/883cb7fa-3eb5-48d4-9cde-7c11307d94f0/64e74d8d-15e7-49a6-a99b-9f52cddf6628"
@@
 		)
 		(instances
+			(project "buck5v"
+				(path "/45bff242-0d9b-4726-901e-ccb01efc2321"
+					(reference "#PWR?")
+					(unit 1)
+				)
+			)
 			(project "doggie_board"
 				(path "/883cb7fa-3eb5-48d4-9cde-7c11307d94f0/64e74d8d-15e7-49a6-a99b-9f52cddf6628"
@@
 		)
 		(instances
+			(project "buck5v"
+				(path "/45bff242-0d9b-4726-901e-ccb01efc2321"
+					(reference "#PWR?")
+					(unit 1)
+				)
+			)
 			(project ""
 				(path "/883cb7fa-3eb5-48d4-9cde-7c11307d94f0/64e74d8d-15e7-49a6-a99b-9f52cddf6628"
@@
 		)
 		(instances
+			(project "buck5v"
+				(path "/45bff242-0d9b-4726-901e-ccb01efc2321"
+					(reference "C?")
+					(unit 1)
+				)
+			)
 			(project "doggie_board"
 				(path "/883cb7fa-3eb5-48d4-9cde-7c11307d94f0/64e74d8d-15e7-49a6-a99b-9f52cddf6628"
@@
 		)
 		(instances
+			(project "buck5v"
+				(path "/45bff242-0d9b-4726-901e-ccb01efc2321"
+					(reference "U?")
+					(unit 1)
+				)
+			)
 			(project ""
 				(path "/883cb7fa-3eb5-48d4-9cde-7c11307d94f0/64e74d8d-15e7-49a6-a99b-9f52cddf6628"
@@
 		)
 		(instances
+			(project "buck5v"
+				(path "/45bff242-0d9b-4726-901e-ccb01efc2321"
+					(reference "#PWR?")
+					(unit 1)
+				)
+			)
 			(project "doggie_board"
 				(path "/883cb7fa-3eb5-48d4-9cde-7c11307d94f0/64e74d8d-15e7-49a6-a99b-9f52cddf6628"
@@
 		)
 		(instances
+			(project "buck5v"
+				(path "/45bff242-0d9b-4726-901e-ccb01efc2321"
+					(reference "C?")
+					(unit 1)
+				)
+			)
 			(project "doggie_board"
 				(path "/883cb7fa-3eb5-48d4-9cde-7c11307d94f0/64e74d8d-15e7-49a6-a99b-9f52cddf6628"
@@
 		)
 		(instances
+			(project "buck5v"
+				(path "/45bff242-0d9b-4726-901e-ccb01efc2321"
+					(reference "R?")
+					(unit 1)
+				)
+			)
 			(project "doggie_board"
 				(path "/883cb7fa-3eb5-48d4-9cde-7c11307d94f0/64e74d8d-15e7-49a6-a99b-9f52cddf6628"
@@
 		)
 		(instances
+			(project "buck5v"
+				(path "/45bff242-0d9b-4726-901e-ccb01efc2321"
+					(reference "C?")
+					(unit 1)
+				)
+			)
 			(project "doggie_board"
 				(path "/883cb7fa-3eb5-48d4-9cde-7c11307d94f0/64e74d8d-15e7-49a6-a99b-9f52cddf6628"
@@
 		)
 		(instances
+			(project "buck5v"
+				(path "/45bff242-0d9b-4726-901e-ccb01efc2321"
+					(reference "C?")
+					(unit 1)
+				)
+			)
 			(project ""
 				(path "/883cb7fa-3eb5-48d4-9cde-7c11307d94f0/64e74d8d-15e7-49a6-a99b-9f52cddf6628"
@@
 		)
 		(instances
+			(project "buck5v"
+				(path "/45bff242-0d9b-4726-901e-ccb01efc2321"
+					(reference "#PWR?")
+					(unit 1)
+				)
+			)
 			(project "doggie_board"
 				(path "/883cb7fa-3eb5-48d4-9cde-7c11307d94f0/64e74d8d-15e7-49a6-a99b-9f52cddf6628"
@@
 		)
 		(instances
+			(project "buck5v"
+				(path "/45bff242-0d9b-4726-901e-ccb01efc2321"
+					(reference "R?")
+					(unit 1)
+				)
+			)
 			(project "doggie_board"
 				(path "/883cb7fa-3eb5-48d4-9cde-7c11307d94f0/64e74d8d-15e7-49a6-a99b-9f52cddf6628"
@@
 		)
 		(instances
+			(project "buck5v"
+				(path "/45bff242-0d9b-4726-901e-ccb01efc2321"
+					(reference "#PWR?")
+					(unit 1)
+				)
+			)
 			(project ""
 				(path "/883cb7fa-3eb5-48d4-9cde-7c11307d94f0/64e74d8d-15e7-49a6-a99b-9f52cddf6628"
@@
 		)
 		(instances
+			(project "buck5v"
+				(path "/45bff242-0d9b-4726-901e-ccb01efc2321"
+					(reference "C?")
+					(unit 1)
+				)
+			)
 			(project "doggie_board"
 				(path "/883cb7fa-3eb5-48d4-9cde-7c11307d94f0/64e74d8d-15e7-49a6-a99b-9f52cddf6628"
@@
 		)
 		(instances
+			(project "buck5v"
+				(path "/45bff242-0d9b-4726-901e-ccb01efc2321"
+					(reference "C?")
+					(unit 1)
+				)
+			)
 			(project "doggie_board"
 				(path "/883cb7fa-3eb5-48d4-9cde-7c11307d94f0/64e74d8d-15e7-49a6-a99b-9f52cddf6628"
@@
 		)
 		(instances
+			(project "buck5v"
+				(path "/45bff242-0d9b-4726-901e-ccb01efc2321"
+					(reference "#PWR?")
+					(unit 1)
+				)
+			)
 			(project "doggie_board"
 				(path "/883cb7fa-3eb5-48d4-9cde-7c11307d94f0/64e74d8d-15e7-49a6-a99b-9f52cddf6628"
@@
 		)
 		(instances
+			(project "buck5v"
+				(path "/45bff242-0d9b-4726-901e-ccb01efc2321"
+					(reference "#PWR?")
+					(unit 1)
+				)
+			)
 			(project "doggie_board"
 				(path "/883cb7fa-3eb5-48d4-9cde-7c11307d94f0/64e74d8d-15e7-49a6-a99b-9f52cddf6628"
@@
 		)
 		(instances
+			(project "buck5v"
+				(path "/45bff242-0d9b-4726-901e-ccb01efc2321"
+					(reference "C?")
+					(unit 1)
+				)
+			)
 			(project ""
 				(path "/883cb7fa-3eb5-48d4-9cde-7c11307d94f0/64e74d8d-15e7-49a6-a99b-9f52cddf6628"
@@
 		)
 		(instances
+			(project "buck5v"
+				(path "/45bff242-0d9b-4726-901e-ccb01efc2321"
+					(reference "C?")
+					(unit 1)
+				)
+			)
 			(project "doggie_board"
 				(path "/883cb7fa-3eb5-48d4-9cde-7c11307d94f0/64e74d8d-15e7-49a6-a99b-9f52cddf6628"
@@
 		)
 		(instances
+			(project "buck5v"
+				(path "/45bff242-0d9b-4726-901e-ccb01efc2321"
+					(reference "#PWR?")
+					(unit 1)
+				)
+			)
 			(project "doggie_board"
 				(path "/883cb7fa-3eb5-48d4-9cde-7c11307d94f0/64e74d8d-15e7-49a6-a99b-9f52cddf6628"
@@
 		)
 		(instances
+			(project "buck5v"
+				(path "/45bff242-0d9b-4726-901e-ccb01efc2321"
+					(reference "#PWR?")
+					(unit 1)
+				)
+			)
 			(project "doggie_board"
 				(path "/883cb7fa-3eb5-48d4-9cde-7c11307d94f0/64e74d8d-15e7-49a6-a99b-9f52cddf6628"
@@
 		)
 		(instances
+			(project "buck5v"
+				(path "/45bff242-0d9b-4726-901e-ccb01efc2321"
+					(reference "#PWR?")
+					(unit 1)
+				)
+			)
 			(project ""
 				(path "/883cb7fa-3eb5-48d4-9cde-7c11307d94f0/64e74d8d-15e7-49a6-a99b-9f52cddf6628"
@@
 		)
 		(instances
+			(project "buck5v"
+				(path "/45bff242-0d9b-4726-901e-ccb01efc2321"
+					(reference "J?")
+					(unit 1)
+				)
+			)
 			(project ""
 				(path "/883cb7fa-3eb5-48d4-9cde-7c11307d94f0/64e74d8d-15e7-49a6-a99b-9f52cddf6628"
@@
 		)
 		(instances
+			(project "buck5v"
+				(path "/45bff242-0d9b-4726-901e-ccb01efc2321"
+					(reference "R?")
+					(unit 1)
+				)
+			)
 			(project "doggie_board"
 				(path "/883cb7fa-3eb5-48d4-9cde-7c11307d94f0/64e74d8d-15e7-49a6-a99b-9f52cddf6628"
@@
 		)
 	)
+	(sheet_instances
+		(path "/"
+			(page "1")
+		)
+	)
+	(embedded_fonts no)
 )

Commit message: fixed footprintns
Parts:
- C10, C11, C12, C13, C14, C15, C16, C17, C18: footprint Capacitor_SMD:C_0201_0603Metric_Pad0.64x0.40mm_HandSolder -> Capacitor_SMD:C_0603_1608Metric_Pad1.08x0.95mm_HandSolder
- R19, R20, R21, R22: footprint Resistor_SMD:R_0201_0603Metric_Pad0.64x0.40mm_HandSolder -> Resistor_SMD:R_0603_1608Metric_Pad0.98x0.95mm_HandSolder
Changed lines of the file:
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@@
 			)
 		)
-		(property "Footprint" "Capacitor_SMD:C_0201_0603Metric_Pad0.64x0.40mm_HandSolder"
+		(property "Footprint" "Capacitor_SMD:C_0603_1608Metric_Pad1.08x0.95mm_HandSolder"
 			(at 120.65 34.29 0)
 			(effects
@@
 			)
 		)
-		(property "Footprint" "Resistor_SMD:R_0201_0603Metric_Pad0.64x0.40mm_HandSolder"
+		(property "Footprint" "Resistor_SMD:R_0603_1608Metric_Pad0.98x0.95mm_HandSolder"
 			(at 22.86 69.85 0)
 			(effects
@@
 			)
 		)
-		(property "Footprint" "Capacitor_SMD:C_0201_0603Metric_Pad0.64x0.40mm_HandSolder"
+		(property "Footprint" "Capacitor_SMD:C_0603_1608Metric_Pad1.08x0.95mm_HandSolder"
 			(at 137.16 34.29 0)
 			(effects
@@
 			)
 		)
-		(property "Footprint" "Capacitor_SMD:C_0201_0603Metric_Pad0.64x0.40mm_HandSolder"
+		(property "Footprint" "Capacitor_SMD:C_0603_1608Metric_Pad1.08x0.95mm_HandSolder"
 			(at 154.94 34.29 0)
 			(effects
@@
 			)
 		)
-		(property "Footprint" "Resistor_SMD:R_0201_0603Metric_Pad0.64x0.40mm_HandSolder"
+		(property "Footprint" "Resistor_SMD:R_0603_1608Metric_Pad0.98x0.95mm_HandSolder"
 			(at 22.86 62.23 0)
 			(effects
@@
 			)
 		)
-		(property "Footprint" "Capacitor_SMD:C_0201_0603Metric_Pad0.64x0.40mm_HandSolder"
+		(property "Footprint" "Capacitor_SMD:C_0603_1608Metric_Pad1.08x0.95mm_HandSolder"
 			(at 146.05 34.29 0)
 			(effects
@@
 			)
 		)
-		(property "Footprint" "Capacitor_SMD:C_0201_0603Metric_Pad0.64x0.40mm_HandSolder"
+		(property "Footprint" "Capacitor_SMD:C_0603_1608Metric_Pad1.08x0.95mm_HandSolder"
 			(at 16.51 36.83 0)
 			(effects
@@
 			)
 		)
-		(property "Footprint" "Resistor_SMD:R_0201_0603Metric_Pad0.64x0.40mm_HandSolder"
+		(property "Footprint" "Resistor_SMD:R_0603_1608Metric_Pad0.98x0.95mm_HandSolder"
 			(at 110.49 41.91 0)
 			(effects
@@
 			)
 		)
-		(property "Footprint" "Capacitor_SMD:C_0201_0603Metric_Pad0.64x0.40mm_HandSolder"
+		(property "Footprint" "Capacitor_SMD:C_0603_1608Metric_Pad1.08x0.95mm_HandSolder"
 			(at 25.4 36.83 0)
 			(effects
@@
 			)
 		)
-		(property "Footprint" "Capacitor_SMD:C_0201_0603Metric_Pad0.64x0.40mm_HandSolder"
+		(property "Footprint" "Capacitor_SMD:C_0603_1608Metric_Pad1.08x0.95mm_HandSolder"
 			(at 34.29 36.83 0)
 			(effects
@@
 			)
 		)
-		(property "Footprint" "Capacitor_SMD:C_0201_0603Metric_Pad0.64x0.40mm_HandSolder"
+		(property "Footprint" "Capacitor_SMD:C_0603_1608Metric_Pad1.08x0.95mm_HandSolder"
 			(at 102.87 34.29 0)
 			(effects
@@
 			)
 		)
-		(property "Footprint" "Capacitor_SMD:C_0201_0603Metric_Pad0.64x0.40mm_HandSolder"
+		(property "Footprint" "Capacitor_SMD:C_0603_1608Metric_Pad1.08x0.95mm_HandSolder"
 			(at 128.27 34.29 0)
 			(effects
@@
 			)
 		)
-		(property "Footprint" "Resistor_SMD:R_0201_0603Metric_Pad0.64x0.40mm_HandSolder"
+		(property "Footprint" "Resistor_SMD:R_0603_1608Metric_Pad0.98x0.95mm_HandSolder"
 			(at 110.49 34.29 0)
 			(effects

Commit message: updated headers
Parts:
- removed J7: Conn_01x03, Connector_PinHeader_2.54mm:PinHeader_1x03_P2.54mm_Vertical, symbol Connector_Generic:Conn_01x03
- removed R19: 100k, Resistor_SMD:R_0603_1608Metric_Pad0.98x0.95mm_HandSolder, symbol Device:R_Small
- removed R20: 20k, Resistor_SMD:R_0603_1608Metric_Pad0.98x0.95mm_HandSolder, symbol Device:R_Small
Other:
- note removed: "Bridge 1 and 2 for always on NMOS adds sequensing (wait for 12V rail good)"
