File: connectors.kicad_sch (KiCad schematic)
At the start: 0 parts

Commit message: Connectors Created
Footprints added
Parts:
- added J5V1, J5V2, J5V3, J5V4, J5V5, J5V6, J5V7, J5V8: Conn_01x02, PinHeader_1x02_P2.54mm_Vertical, symbol Connector_Generic:Conn_01x02
- added J5V10, J5V11, J5V12, J5V13, J5V14, J5V15, J5V16, J5V17, J5V18, J5V9: Conn_01x02, XT30PW-M:AMASS_XT30PW-M, symbol Connector_Generic:Conn_01x02
Connections:
- new net +3.3V: J5V5.1 (Pin_1), J5V6.1 (Pin_1), J5V7.1 (Pin_1), J5V8.1 (Pin_1)
- new net +48V: J5V10.1 (Pin_1), J5V11.1 (Pin_1), J5V12.1 (Pin_1), J5V13.1 (Pin_1), J5V14.1 (Pin_1), J5V15.1 (Pin_1), J5V16.1 (Pin_1), J5V17.1 (Pin_1), J5V18.1 (Pin_1), J5V9.1 (Pin_1)
- new net +5V: J5V1.1 (Pin_1), J5V2.1 (Pin_1), J5V3.1 (Pin_1), J5V4.1 (Pin_1)
- new net GND: J5V1.2 (Pin_2), J5V10.2 (Pin_2), J5V11.2 (Pin_2), J5V12.2 (Pin_2), J5V13.2 (Pin_2), J5V14.2 (Pin_2), J5V15.2 (Pin_2), J5V16.2 (Pin_2), J5V17.2 (Pin_2), J5V18.2 (Pin_2), J5V2.2 (Pin_2), J5V3.2 (Pin_2), J5V4.2 (Pin_2), J5V5.2 (Pin_2), J5V6.2 (Pin_2), J5V7.2 (Pin_2), J5V8.2 (Pin_2), J5V9.2 (Pin_2)

Commit message: Renaming of Parts
Rename
Other:
- company: (none) -> UMass Robotics
- title: (none) -> Connectors
Changed lines of the file:
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@@
 	(generator_version "9.0")
 	(paper "A4")
+	(title_block
+		(title "Connectors")
+		(company "UMass Robotics")
+		(comment 2 "Niranjan Mathirajan")
+		(comment 3 "Alperen Ozpolat")
+	)
 	(symbol
 		(lib_id "power:GND")

Commit message: updated footprints and pcb
Parts:
- added J5V19, J5V20: Conn_01x02, Connector_AMASS:AMASS_XT30U-F_1x02_P5.0mm_Vertical, symbol Connector_Generic:Conn_01x02
- J5V10, J5V11, J5V12, J5V13, J5V14, J5V9: footprint XT30PW-M:AMASS_XT30PW-M -> Connector_AMASS:AMASS_XT30PW-F_1x02_P2.50mm_Horizontal
- J5V15, J5V16, J5V17, J5V18: footprint XT30PW-M:AMASS_XT30PW-M -> Connector_AMASS:AMASS_XT30U-F_1x02_P5.0mm_Vertical
Connections:
- net +48V: now also J5V19.1 (Pin_1), J5V20.1 (Pin_1)
- net GND: now also J5V19.2 (Pin_2), J5V20.2 (Pin_2)

Commit message: updates
Parts:
- removed J5V10, J5V11, J5V13, J5V14: Conn_01x02, Connector_AMASS:AMASS_XT30PW-F_1x02_P2.50mm_Horizontal, symbol Connector_Generic:Conn_01x02
- added J5V4, J5V5, J5V7, J5V8: Conn_01x02, Connector_AMASS:AMASS_XT30U-F_1x02_P5.0mm_Vertical, symbol Connector_Generic:Conn_01x02
- J5V12, J5V9: footprint Connector_AMASS:AMASS_XT30PW-F_1x02_P2.50mm_Horizontal -> Connector_AMASS:AMASS_XT30U-F_1x02_P5.0mm_Vertical
- renumbered J5V16 to J5V1, J5V20 to J5V10, J5V19 to J5V11, J5V6 to J5V13, J5V7 to J5V14, J5V8 to J5V15, J5V5 to J5V16, J5V1 to J5V17, J5V2 to J5V18, J5V3 to J5V19, J5V17 to J5V2, J5V4 to J5V20, J5V18 to J5V3, J5V15 to J5V6
Connections:
- net GND: now also J5V4.2 (Pin_2), J5V5.2 (Pin_2), J5V7.2 (Pin_2), J5V8.2 (Pin_2)
- net +48V renamed 48v_switched
- net 48v_switched: now also J5V4.1 (Pin_1), J5V5.1 (Pin_1), J5V7.1 (Pin_1), J5V8.1 (Pin_1)
Other:
- moved on the sheet: J5V1, J5V10, J5V11, J5V13, J5V14, J5V15, J5V16, J5V17, J5V18, J5V19, J5V2, J5V20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

Commit message: fixed ERC
Parts:
- J5V1, J5V10, J5V11, J5V12, J5V2, J5V3, J5V4, J5V5, J5V6, J5V7, J5V8, J5V9: footprint Connector_AMASS:AMASS_XT30U-F_1x02_P5.0mm_Vertical -> Connector_AMASS:AMASS_XT30PW-M_1x02_P2.50mm_Horizontal
- J5V13, J5V14, J5V15, J5V16, J5V17, J5V18, J5V19, J5V20: footprint PinHeader_1x02_P2.54mm_Vertical -> Connector_PinHeader_1.00mm:PinHeader_1x02_P1.00mm_Vertical
Connections:
- net 48v_switched: no longer J5V1.1 (Pin_1), J5V10.1 (Pin_1), J5V11.1 (Pin_1), J5V2.1 (Pin_1), J5V3.1 (Pin_1), J5V4.1 (Pin_1), J5V5.1 (Pin_1), J5V7.1 (Pin_1), J5V8.1 (Pin_1), J5V9.1 (Pin_1)
- new net +48V: J5V1.1 (Pin_1), J5V10.1 (Pin_1), J5V11.1 (Pin_1), J5V2.1 (Pin_1), J5V3.1 (Pin_1), J5V4.1 (Pin_1), J5V5.1 (Pin_1), J5V7.1 (Pin_1), J5V8.1 (Pin_1), J5V9.1 (Pin_1)

Commit message: routing progress
Connections:
- net 48v_switched is gone; now on net +48V: J5V12.1 (Pin_1), J5V6.1 (Pin_1)

Commit message: Fixed Schematics with more cost effective IC's
Parts:
- added J5V13: Conn_01x02, Connector_BarrelJack:BarrelJack_CUI_PJ-079BH_Horizontal, symbol Connector_Generic:Conn_01x02
- added J5V14, J5V15, J5V16: Conn_01x02, Connector_PinHeader_1.00mm:PinHeader_1x02_P1.00mm_Vertical, symbol Connector_Generic:Conn_01x02
- J5V21: renamed from J5V17; footprint Connector_PinHeader_1.00mm:PinHeader_1x02_P1.00mm_Vertical -> Connector_BarrelJack:BarrelJack_CUI_PJ-079BH_Horizontal
- renumbered J5V13 to J5V17, J5V14 to J5V18, J5V15 to J5V19, J5V16 to J5V20, J5V18 to J5V22, J5V19 to J5V23, J5V20 to J5V24
Connections:
- net GND: now also J5V13.2 (Pin_2), J5V14.2 (Pin_2), J5V15.2 (Pin_2), J5V16.2 (Pin_2)
- new net +12V: J5V13.1 (Pin_1), J5V14.1 (Pin_1), J5V15.1 (Pin_1), J5V16.1 (Pin_1)
Other:
- moved on the sheet: J5V1, J5V10, J5V11, J5V12, J5V2, J5V21, J5V22, J5V23, J5V24, J5V3, J5V4, J5V5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
