File: connectors.kicad_sch (KiCad schematic)
At the start: 24 parts, among them J5V1 Conn_01x02, J5V10 Conn_01x02, J5V11 Conn_01x02, J5V12 Conn_01x02, J5V13 Conn_01x02, J5V14 Conn_01x02, J5V15 Conn_01x02, J5V16 Conn_01x02, J5V17 Conn_01x02, J5V18 Conn_01x02, J5V19 Conn_01x02, J5V2 Conn_01x02, J5V20 Conn_01x02, J5V21 Conn_01x02, J5V22 Conn_01x02, J5V23 Conn_01x02, J5V24 Conn_01x02, J5V3 Conn_01x02, J5V4 Conn_01x02, J5V5 Conn_01x02, J5V6 Conn_01x02, J5V7 Conn_01x02, J5V8 Conn_01x02, J5V9 Conn_01x02

Commit message: pcb routing
Parts:
- J5V1, J5V10, J5V11, J5V12, J5V2, J5V3, J5V4, J5V5, J5V6, J5V7, J5V8, J5V9: value Conn_01x02 -> 48v
- J5V13: value Conn_01x02 -> 12v
- J5V14, J5V15, J5V16: value Conn_01x02 -> 12v; footprint Connector_PinHeader_1.00mm:PinHeader_1x02_P1.00mm_Vertical -> Connector_PinHeader_2.54mm:PinHeader_1x02_P2.54mm_Vertical
- J5V17, J5V18, J5V19, J5V20: value Conn_01x02 -> 3.3v; footprint Connector_PinHeader_1.00mm:PinHeader_1x02_P1.00mm_Vertical -> Connector_PinHeader_2.54mm:PinHeader_1x02_P2.54mm_Vertical
- J5V21: value Conn_01x02 -> 5v
- J5V22, J5V23, J5V24: value Conn_01x02 -> 5v; footprint Connector_PinHeader_1.00mm:PinHeader_1x02_P1.00mm_Vertical -> Connector_PinHeader_2.54mm:PinHeader_1x02_P2.54mm_Vertical
Changed lines of the file:
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@@
 			)
 		)
-		(property "Value" "Conn_01x02"
+		(property "Value" "3.3v"
 			(at 125.73 25.3999 90)
 			(effects
@@
 			)
 		)
-		(property "Footprint" "Connector_PinHeader_1.00mm:PinHeader_1x02_P1.00mm_Vertical"
+		(property "Footprint" "Connector_PinHeader_2.54mm:PinHeader_1x02_P2.54mm_Vertical"
 			(at 123.19 24.13 0)
 			(effects
@@
 			)
 		)
-		(property "Value" "Conn_01x02"
+		(property "Value" "48v"
 			(at 21.59 40.6399 90)
 			(effects
@@
 			)
 		)
-		(property "Value" "Conn_01x02"
+		(property "Value" "48v"
 			(at 45.72 40.6399 90)
 			(effects
@@
 			)
 		)
-		(property "Value" "Conn_01x02"
+		(property "Value" "48v"
 			(at 45.72 68.5799 90)
 			(effects
@@
 			)
 		)
-		(property "Value" "Conn_01x02"
+		(property "Value" "5v"
 			(at 149.86 26.6699 90)
 			(effects
@@
 			)
 		)
-		(property "Value" "Conn_01x02"
+		(property "Value" "48v"
 			(at 21.59 82.5499 90)
 			(effects
@@
 			)
 		)
-		(property "Value" "Conn_01x02"
+		(property "Value" "48v"
 			(at 45.72 82.5499 90)
 			(effects
@@
 			)
 		)
-		(property "Value" "Conn_01x02"
+		(property "Value" "3.3v"
 			(at 125.73 67.3099 90)
 			(effects
@@
 			)
 		)
-		(property "Footprint" "Connector_PinHeader_1.00mm:PinHeader_1x02_P1.00mm_Vertical"
+		(property "Footprint" "Connector_PinHeader_2.54mm:PinHeader_1x02_P2.54mm_Vertical"
 			(at 123.19 66.04 0)
 			(effects
@@
 			)
 		)
-		(property "Value" "Conn_01x02"
+		(property "Value" "3.3v"
 			(at 125.73 53.3399 90)
 			(effects
@@
 			)
 		)
-		(property "Footprint" "Connector_PinHeader_1.00mm:PinHeader_1x02_P1.00mm_Vertical"
+		(property "Footprint" "Connector_PinHeader_2.54mm:PinHeader_1x02_P2.54mm_Vertical"
 			(at 123.19 52.07 0)
 			(effects
@@
 			)
 		)
-		(property "Value" "Conn_01x02"
+		(property "Value" "48v"
 			(at 21.59 96.5199 90)
 			(effects
@@
 			)
 		)
-		(property "Value" "Conn_01x02"
+		(property "Value" "48v"
 			(at 45.72 96.5199 90)
 			(effects
@@
 			)
 		)
-		(property "Value" "Conn_01x02"
+		(property "Value" "5v"
 			(at 149.86 59.6899 90)
 			(effects
@@
 			)
 		)
-		(property "Footprint" "Connector_PinHeader_1.00mm:PinHeader_1x02_P1.00mm_Vertical"
+		(property "Footprint" "Connector_PinHeader_2.54mm:PinHeader_1x02_P2.54mm_Vertical"
 			(at 147.32 58.42 0)
 			(effects
@@
 			)
 		)
-		(property "Value" "Conn_01x02"
+		(property "Value" "48v"
 			(at 21.59 68.5799 90)
 			(effects
@@
 			)
 		)
-		(property "Value" "Conn_01x02"
+		(property "Value" "5v"
 			(at 149.86 41.9099 90)
 			(effects
@@
 			)
 		)
-		(property "Footprint" "Connector_PinHeader_1.00mm:PinHeader_1x02_P1.00mm_Vertical"
+		(property "Footprint" "Connector_PinHeader_2.54mm:PinHeader_1x02_P2.54mm_Vertical"
 			(at 147.32 40.64 0)
 			(effects
@@
 			)
 		)
-		(property "Value" "Conn_01x02"
+		(property "Value" "12v"
 			(at 73.66 27.9399 90)
 			(effects
@@
 			)
 		)
-		(property "Value" "Conn_01x02"
+		(property "Value" "48v"
 			(at 21.59 26.6699 90)
 			(effects
@@
 			)
 		)
-		(property "Value" "Conn_01x02"
+		(property "Value" "48v"
 			(at 45.72 26.6699 90)
 			(effects
@@
 			)
 		)
-		(property "Value" "Conn_01x02"
+		(property "Value" "3.3v"
 			(at 125.73 39.3699 90)
 			(effects
@@
 			)
 		)
-		(property "Footprint" "Connector_PinHeader_1.00mm:PinHeader_1x02_P1.00mm_Vertical"
+		(property "Footprint" "Connector_PinHeader_2.54mm:PinHeader_1x02_P2.54mm_Vertical"
 			(at 123.19 38.1 0)
 			(effects
@@
 			)
 		)
-		(property "Value" "Conn_01x02"
+		(property "Value" "12v"
 			(at 73.66 76.1999 90)
 			(effects
@@
 			)
 		)
-		(property "Footprint" "Connector_PinHeader_1.00mm:PinHeader_1x02_P1.00mm_Vertical"
+		(property "Footprint" "Connector_PinHeader_2.54mm:PinHeader_1x02_P2.54mm_Vertical"
 			(at 71.12 74.93 0)
 			(effects
@@
 			)
 		)
-		(property "Value" "Conn_01x02"
+		(property "Value" "12v"
 			(at 73.66 43.1799 90)
 			(effects
@@
 			)
 		)
-		(property "Footprint" "Connector_PinHeader_1.00mm:PinHeader_1x02_P1.00mm_Vertical"
+		(property "Footprint" "Connector_PinHeader_2.54mm:PinHeader_1x02_P2.54mm_Vertical"
 			(at 71.12 41.91 0)
 			(effects
@@
 			)
 		)
-		(property "Value" "Conn_01x02"
+		(property "Value" "12v"
 			(at 73.66 60.9599 90)
 			(effects
@@
 			)
 		)
-		(property "Footprint" "Connector_PinHeader_1.00mm:PinHeader_1x02_P1.00mm_Vertical"
+		(property "Footprint" "Connector_PinHeader_2.54mm:PinHeader_1x02_P2.54mm_Vertical"
 			(at 71.12 59.69 0)
 			(effects
@@
 			)
 		)
-		(property "Value" "Conn_01x02"
+		(property "Value" "5v"
 			(at 149.86 74.9299 90)
 			(effects
@@
 			)
 		)
-		(property "Footprint" "Connector_PinHeader_1.00mm:PinHeader_1x02_P1.00mm_Vertical"
+		(property "Footprint" "Connector_PinHeader_2.54mm:PinHeader_1x02_P2.54mm_Vertical"
 			(at 147.32 73.66 0)
 			(effects
@@
 			)
 		)
-		(property "Value" "Conn_01x02"
+		(property "Value" "48v"
 			(at 21.59 54.6099 90)
 			(effects
@@
 			)
 		)
-		(property "Value" "Conn_01x02"
+		(property "Value" "48v"
 			(at 45.72 54.6099 90)
 			(effects

Commit message: shortened board
Parts:
- J5V13, J5V21: footprint Connector_BarrelJack:BarrelJack_CUI_PJ-079BH_Horizontal -> footprints:CUI_PJ-037A
Changed lines of the file:
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@@
 			)
 		)
-		(property "Footprint" "Connector_BarrelJack:BarrelJack_CUI_PJ-079BH_Horizontal"
+		(property "Footprint" "footprints:CUI_PJ-037A"
 			(at 147.32 25.4 0)
 			(effects
@@
 			)
 		)
-		(property "Footprint" "Connector_BarrelJack:BarrelJack_CUI_PJ-079BH_Horizontal"
+		(property "Footprint" "footprints:CUI_PJ-037A"
 			(at 71.12 26.67 0)
 			(effects

Commit message: updated headers
Parts:
- removed J5V14, J5V15, J5V16: 12v, Connector_PinHeader_2.54mm:PinHeader_1x02_P2.54mm_Vertical, symbol Connector_Generic:Conn_01x02
- removed J5V17, J5V18, J5V19, J5V20: 3.3v, Connector_PinHeader_2.54mm:PinHeader_1x02_P2.54mm_Vertical, symbol Connector_Generic:Conn_01x02
- removed J5V22, J5V23, J5V24: 5v, Connector_PinHeader_2.54mm:PinHeader_1x02_P2.54mm_Vertical, symbol Connector_Generic:Conn_01x02
- added J1: Conn_02x08_Odd_Even, Connector_PinHeader_2.54mm:PinHeader_2x08_P2.54mm_Vertical, symbol Connector_Generic:Conn_02x08_Odd_Even
- added J10, J9: Conn_02x04_Odd_Even, Connector_PinHeader_2.54mm:PinHeader_2x04_P2.54mm_Vertical, symbol Connector_Generic:Conn_02x04_Odd_Even
- added J12: Conn_02x05_Odd_Even, Connector_PinHeader_2.54mm:PinHeader_2x05_P2.54mm_Vertical, symbol Connector_Generic:Conn_02x05_Odd_Even
Connections:
- net +12V: now also J9.1 (Pin_1), J9.3 (Pin_3), J9.5 (Pin_5), J9.7 (Pin_7)
- net +3.3V: now also J12.1 (Pin_1), J12.3 (Pin_3), J12.5 (Pin_5), J12.7 (Pin_7), J12.9 (Pin_9)
- net +5V: now also J10.1 (Pin_1), J10.3 (Pin_3), J10.5 (Pin_5), J10.7 (Pin_7)
- net GND: now also J1.10 (Pin_10), J1.12 (Pin_12), J1.14 (Pin_14), J1.16 (Pin_16), J1.2 (Pin_2), J1.4 (Pin_4), J1.6 (Pin_6), J1.8 (Pin_8), J10.2 (Pin_2), J10.4 (Pin_4), J10.6 (Pin_6), J10.8 (Pin_8), J12.10 (Pin_10), J12.2 (Pin_2), J12.4 (Pin_4), J12.6 (Pin_6), J12.8 (Pin_8), J9.2 (Pin_2), J9.4 (Pin_4), J9.6 (Pin_6), J9.8 (Pin_8)
- new net +3.3V_LP: J1.1 (Pin_1), J1.15 (Pin_15)
- new net 12V_EN: J1.13 (Pin_13)
- new net 12V_PG: J1.5 (Pin_5)
- new net 3V3_EN: J1.9 (Pin_9)
- new net 48V_EN: J1.7 (Pin_7)
- new net 48V_PG: J1.3 (Pin_3)
- new net 5V_EN: J1.11 (Pin_11)
