File: untitled.kicad_sch (KiCad schematic)
At the start: 11 parts, among them U4 LM76005

Commit message: updates
Parts:
- renumbered Cboot to Cboot3, Cin to Cin3, Cinx to Cinx3, Cout to Cout3, Coutx to Coutx3, Cvcc to Cvcc3, L1(2) to L1(2)1, Rfbb to Rfbb3, Rfbt to Rfbt3, Rpgood to Rpgood3
Connections:
- net V_switched renamed 48v_switched
Changed lines of the file:
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@@
 		)
 	)
-	(global_label "V_switched"
+	(global_label "48v_switched"
 		(shape input)
 		(at 49.53 57.15 180)
@@
 		)
 		(property "Intersheetrefs" "${INTERSHEET_REFS}"
-			(at 36.3243 57.15 0)
+			(at 34.0263 57.15 0)
 			(effects
 				(font
@@
 		(dnp no)
 		(fields_autoplaced yes)
-		(property "Reference" "Rfbt"
+		(property "Reference" "Rfbt3"
 			(at 217.17 69.8499 0)
 			(effects
@@
 			(project ""
 				(path "/883cb7fa-3eb5-48d4-9cde-7c11307d94f0/c35c9e48-520d-4065-aa61-8aea5a619a4f"
-					(reference "Rfbt")
+					(reference "Rfbt3")
 					(unit 1)
 				)
@@
 		(dnp no)
 		(fields_autoplaced yes)
-		(property "Reference" "L1(2)"
+		(property "Reference" "L1(2)1"
 			(at 191.77 45.72 90)
 			(effects
@@
 			(project ""
 				(path "/883cb7fa-3eb5-48d4-9cde-7c11307d94f0/c35c9e48-520d-4065-aa61-8aea5a619a4f"
-					(reference "L1(2)")
+					(reference "L1(2)1")
 					(unit 1)
 				)
@@
 		(dnp no)
 		(fields_autoplaced yes)
-		(property "Reference" "Cboot"
+		(property "Reference" "Cboot3"
 			(at 167.64 64.7699 0)
 			(effects
@@
 			(project ""
 				(path "/883cb7fa-3eb5-48d4-9cde-7c11307d94f0/c35c9e48-520d-4065-aa61-8aea5a619a4f"
-					(reference "Cboot")
+					(reference "Cboot3")
 					(unit 1)
 				)
@@
 		(dnp no)
 		(fields_autoplaced yes)
-		(property "Reference" "Cvcc"
+		(property "Reference" "Cvcc3"
 			(at 166.37 95.2499 0)
 			(effects
@@
 			(project ""
 				(path "/883cb7fa-3eb5-48d4-9cde-7c11307d94f0/c35c9e48-520d-4065-aa61-8aea5a619a4f"
-					(reference "Cvcc")
+					(reference "Cvcc3")
 					(unit 1)
 				)
@@
 		(on_board yes)
 		(dnp no)
-		(property "Reference" "Cin"
+		(property "Reference" "Cin3"
 			(at 53.34 78.7399 0)
 			(effects
@@
 			(project ""
 				(path "/883cb7fa-3eb5-48d4-9cde-7c11307d94f0/c35c9e48-520d-4065-aa61-8aea5a619a4f"
-					(reference "Cin")
+					(reference "Cin3")
 					(unit 1)
 				)
@@
 		(dnp no)
 		(fields_autoplaced yes)
-		(property "Reference" "Rpgood"
+		(property "Reference" "Rpgood3"
 			(at 111.76 35.56 90)
 			(effects
@@
 			(project ""
 				(path "/883cb7fa-3eb5-48d4-9cde-7c11307d94f0/c35c9e48-520d-4065-aa61-8aea5a619a4f"
-					(reference "Rpgood")
+					(reference "Rpgood3")
 					(unit 1)
 				)
@@
 		(on_board yes)
 		(dnp no)
-		(property "Reference" "Coutx"
+		(property "Reference" "Coutx3"
 			(at 270.51 78.7399 0)
 			(effects
@@
 			(project ""
 				(path "/883cb7fa-3eb5-48d4-9cde-7c11307d94f0/c35c9e48-520d-4065-aa61-8aea5a619a4f"
-					(reference "Coutx")
+					(reference "Coutx3")
 					(unit 1)
 				)
@@
 		(dnp no)
 		(fields_autoplaced yes)
-		(property "Reference" "Cinx"
+		(property "Reference" "Cinx3"
 			(at 73.66 78.7399 0)
 			(effects
@@
 			(project ""
 				(path "/883cb7fa-3eb5-48d4-9cde-7c11307d94f0/c35c9e48-520d-4065-aa61-8aea5a619a4f"
-					(reference "Cinx")
+					(reference "Cinx3")
 					(unit 1)
 				)
@@
 		(dnp no)
 		(fields_autoplaced yes)
-		(property "Reference" "Rfbb"
+		(property "Reference" "Rfbb3"
 			(at 217.17 90.1699 0)
 			(effects
@@
 			(project ""
 				(path "/883cb7fa-3eb5-48d4-9cde-7c11307d94f0/c35c9e48-520d-4065-aa61-8aea5a619a4f"
-					(reference "Rfbb")
+					(reference "Rfbb3")
 					(unit 1)
 				)
@@
 		(dnp no)
 		(fields_autoplaced yes)
-		(property "Reference" "Cout"
+		(property "Reference" "Cout3"
 			(at 241.3 78.1049 0)
 			(effects
@@
 			(project ""
 				(path "/883cb7fa-3eb5-48d4-9cde-7c11307d94f0/c35c9e48-520d-4065-aa61-8aea5a619a4f"
-					(reference "Cout")
-					(unit 1)
-				)
+					(reference "Cout3")
+					(unit 1)
+				)

Commit message: Connectors Created
Footprints added
Parts:
- Cboot3, Cinx3, Cout3, Coutx3, Cvcc3: footprint (none) -> Capacitor_SMD:C_0805_2012Metric_Pad1.18x1.45mm_HandSolder
- L1(2)1: footprint (none) -> Inductor_SMD:L_6.3x6.3_H3
- Rfbb3, Rfbt3, Rpgood3: footprint (none) -> Resistor_SMD:R_0201_0603Metric
Changed lines of the file:
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@@
 			)
 		)
-		(property "Footprint" ""
+		(property "Footprint" "Resistor_SMD:R_0201_0603Metric"
 			(at 212.852 71.12 90)
 			(effects
@@
 			)
 		)
-		(property "Footprint" ""
+		(property "Footprint" "Inductor_SMD:L_6.3x6.3_H3"
 			(at 191.77 50.8 0)
 			(effects
@@
 			)
 		)
-		(property "Footprint" ""
+		(property "Footprint" "Capacitor_SMD:C_0805_2012Metric_Pad1.18x1.45mm_HandSolder"
 			(at 164.7952 69.85 0)
 			(effects
@@
 			)
 		)
-		(property "Footprint" ""
+		(property "Footprint" "Capacitor_SMD:C_0805_2012Metric_Pad1.18x1.45mm_HandSolder"
 			(at 163.5252 100.33 0)
 			(effects
@@
 			)
 		)
-		(property "Footprint" ""
+		(property "Footprint" "Resistor_SMD:R_0201_0603Metric"
 			(at 111.76 40.132 90)
 			(effects
@@
 			)
 		)
-		(property "Footprint" ""
+		(property "Footprint" "Capacitor_SMD:C_0805_2012Metric_Pad1.18x1.45mm_HandSolder"
 			(at 267.6652 83.82 0)
 			(effects
@@
 			)
 		)
-		(property "Footprint" ""
+		(property "Footprint" "Capacitor_SMD:C_0805_2012Metric_Pad1.18x1.45mm_HandSolder"
 			(at 70.8152 83.82 0)
 			(effects
@@
 			)
 		)
-		(property "Footprint" ""
+		(property "Footprint" "Resistor_SMD:R_0201_0603Metric"
 			(at 212.852 91.44 90)
 			(effects
@@
 			)
 		)
-		(property "Footprint" ""
+		(property "Footprint" "Capacitor_SMD:C_0805_2012Metric_Pad1.18x1.45mm_HandSolder"
 			(at 237.49 80.01 0)
 			(effects

Commit message: Renaming of Parts
Rename
Parts:
- Rfbb3: value 43.2kOhm -> 43.2k
- Rfbt3, Rpgood3: value 100kOhm -> 100k
Other:
- company: (none) -> UMass Robotics
- title: (none) -> 48v to 3.3v Converter
Changed lines of the file:
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@@
 	(generator_version "9.0")
 	(paper "A4")
+	(title_block
+		(title "48v to 3.3v Converter")
+		(company "UMass Robotics")
+		(comment 2 "Niranjan Mathirajan")
+		(comment 3 "Alperen Ozpolat")
+	)
 	(junction
 		(at 69.85 57.15)
@@
 			)
 		)
-		(property "Value" "100kOhm"
+		(property "Value" "100k"
 			(at 217.17 72.3899 0)
 			(effects
@@
 			)
 		)
-		(property "Value" "100kOhm"
+		(property "Value" "100k"
 			(at 111.76 38.1 90)
 			(effects
@@
 			)
 		)
-		(property "Value" "43.2kOhm"
+		(property "Value" "43.2k"
 			(at 217.17 92.7099 0)
 			(effects

Commit message: updates
Parts:
- renumbered U4 to U5
Changed lines of the file:
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@@
 		(dnp no)
 		(fields_autoplaced yes)
-		(property "Reference" "#PWR015"
+		(property "Reference" "#PWR058"
 			(at 142.24 110.49 0)
 			(effects
@@
 			(project ""
 				(path "/883cb7fa-3eb5-48d4-9cde-7c11307d94f0/c35c9e48-520d-4065-aa61-8aea5a619a4f"
-					(reference "#PWR015")
+					(reference "#PWR058")
 					(unit 1)
 				)
@@
 		(dnp no)
 		(fields_autoplaced yes)
-		(property "Reference" "#FLG04"
+		(property "Reference" "#FLG08"
 			(at 270.51 47.625 0)
 			(effects
@@
 			(project "doggie_board"
 				(path "/883cb7fa-3eb5-48d4-9cde-7c11307d94f0/c35c9e48-520d-4065-aa61-8aea5a619a4f"
-					(reference "#FLG04")
+					(reference "#FLG08")
 					(unit 1)
 				)
@@
 		(dnp no)
 		(fields_autoplaced yes)
-		(property "Reference" "#PWR019"
+		(property "Reference" "#PWR060"
 			(at 162.56 106.68 0)
 			(effects
@@
 			(project ""
 				(path "/883cb7fa-3eb5-48d4-9cde-7c11307d94f0/c35c9e48-520d-4065-aa61-8aea5a619a4f"
-					(reference "#PWR019")
+					(reference "#PWR060")
 					(unit 1)
 				)
@@
 		(dnp no)
 		(fields_autoplaced yes)
-		(property "Reference" "#PWR020"
+		(property "Reference" "#PWR061"
 			(at 278.13 54.61 0)
 			(effects
@@
 			(project "doggie_board"
 				(path "/883cb7fa-3eb5-48d4-9cde-7c11307d94f0/c35c9e48-520d-4065-aa61-8aea5a619a4f"
-					(reference "#PWR020")
+					(reference "#PWR061")
 					(unit 1)
 				)
@@
 		(dnp no)
 		(fields_autoplaced yes)
-		(property "Reference" "U4"
+		(property "Reference" "U5"
 			(at 138.43 55.88 0)
 			(effects
@@
 			(project "doggie_board"
 				(path "/883cb7fa-3eb5-48d4-9cde-7c11307d94f0/c35c9e48-520d-4065-aa61-8aea5a619a4f"
-					(reference "U4")
+					(reference "U5")
 					(unit 1)
 				)
@@
 		(dnp no)
 		(fields_autoplaced yes)
-		(property "Reference" "#PWR016"
+		(property "Reference" "#PWR059"
 			(at 157.48 50.8 0)
 			(effects
@@
 			(project ""
 				(path "/883cb7fa-3eb5-48d4-9cde-7c11307d94f0/c35c9e48-520d-4065-aa61-8aea5a619a4f"
-					(reference "#PWR016")
+					(reference "#PWR059")
 					(unit 1)
 				)
@@
 		(dnp no)
 		(fields_autoplaced yes)
-		(property "Reference" "#FLG05"
+		(property "Reference" "#FLG07"
 			(at 59.69 55.245 0)
 			(effects
@@
 			(project "doggie_board"
 				(path "/883cb7fa-3eb5-48d4-9cde-7c11307d94f0/c35c9e48-520d-4065-aa61-8aea5a619a4f"
-					(reference "#FLG05")
-					(unit 1)
-				)
+					(reference "#FLG07")
+					(unit 1)
+				)

Commit message: fixed ERC
Connections:
- net 48v_switched renamed +48V
Changed lines of the file:
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@@
+	)
+	(junction
+		(at 50.8 57.15)
+		(diameter 0)
+		(color 0 0 0 0)
 	)
 	(junction
@@
 	(wire
 		(pts
-			(xy 59.69 57.15) (xy 49.53 57.15)
+			(xy 59.69 57.15) (xy 50.8 57.15)
 		)
 		(stroke
@@
 	(wire
 		(pts
+			(xy 50.8 57.15) (xy 49.53 57.15)
+		)
+		(stroke
+			(width 0)
+			(type default)
+		)
+	)
+	(wire
+		(pts
 			(xy 214.63 80.01) (xy 214.63 87.63)
 		)
@@
 			(width 0)
 			(type default)
-		)
-	)
-	(global_label "48v_switched"
-		(shape input)
-		(at 49.53 57.15 180)
-		(fields_autoplaced yes)
-		(effects
-			(font
-				(size 1.27 1.27)
-			)
-			(justify right)
-		)
-		(property "Intersheetrefs" "${INTERSHEET_REFS}"
-			(at 34.0263 57.15 0)
-			(effects
-				(font
-					(size 1.27 1.27)
-				)
-				(justify right)
-				(hide yes)
-			)
 		)
 	)
@@
 					(unit 1)
 				)
+			)
+		)
+	)
+	(symbol
+		(lib_id "power:+48V")
+		(at 50.8 57.15 0)
+		(unit 1)
+		(exclude_from_sim no)
+		(in_bom yes)
+		(on_board yes)
+		(dnp no)
+		(fields_autoplaced yes)
+		(property "Reference" "#PWR063"
+			(at 50.8 60.96 0)
+			(effects
+				(font
+					(size 1.27 1.27)
+				)
+				(hide yes)
+			)
+		)
+		(property "Value" "+48V"
+			(at 50.8 52.07 0)
+			(effects
+				(font
+					(size 1.27 1.27)
+				)
+			)
+		)
+		(property "Footprint" ""
+			(at 50.8 57.15 0)
+			(effects
+				(font
+					(size 1.27 1.27)
+				)
+				(hide yes)
+			)
+		)
+		(property "Datasheet" ""
+			(at 50.8 57.15 0)
+			(effects
+				(font
+					(size 1.27 1.27)
+				)
+				(hide yes)
+			)
+		)
+		(property "Description" "Power symbol creates a global label with name \"+48V\""
+			(at 50.8 57.15 0)
+			(effects
+				(font
+					(size 1.27 1.27)
+				)
+				(hide yes)
+			)
+		)
+		(pin "1"
+		)
+		(instances
+			(project "doggie_board"
+				(path "/883cb7fa-3eb5-48d4-9cde-7c11307d94f0/c35c9e48-520d-4065-aa61-8aea5a619a4f"
+					(reference "#PWR063")
+					(unit 1)
+				)

Commit message: Fixed Schematics with more cost effective IC's
Parts:
- removed Cboot3: 470nF, 20mOhm, Capacitor_SMD:C_0805_2012Metric_Pad1.18x1.45mm_HandSolder, symbol Device:C
- removed Cin3: 4.7 uF, 5.89 mOhm, symbol Device:C
- removed Cinx3: 470nF, 33.996mOhm, Capacitor_SMD:C_0805_2012Metric_Pad1.18x1.45mm_HandSolder, symbol Device:C
- removed Cout3: 220uF, 10 mOhm, Capacitor_SMD:C_0805_2012Metric_Pad1.18x1.45mm_HandSolder, symbol Device:C_Polarized_US
- removed Coutx3: 470nF, 58.782mOhm, Capacitor_SMD:C_0805_2012Metric_Pad1.18x1.45mm_HandSolder, symbol Device:C
- removed Cvcc3: 2.2uF, 7.474mOhm, Capacitor_SMD:C_0805_2012Metric_Pad1.18x1.45mm_HandSolder, symbol Device:C
- removed L1(2)1: 4.7uH, 13.1mOhm, Inductor_SMD:L_6.3x6.3_H3, symbol Device:L
- removed Rfbb3: 43.2k, Resistor_SMD:R_0201_0603Metric, symbol Device:R
- removed Rfbt3, Rpgood3: 100k, Resistor_SMD:R_0201_0603Metric, symbol Device:R
- removed U5: LM76005, Package_DFN_QFN:Texas_RNP0030B_WQFN-30-1EP_4x6mm_P0.5mm_EP1.8x4.5mm, symbol Regulator_Switching:LM76005
- added C19, C20: 10u, symbol Device:C_Small
- added C21, C27: 100n, symbol Device:C_Small
- added C22: 56p, symbol Device:C_Small
- added C23, C24, C25, C26: 22u, symbol Device:C_Small
- added L3: 2.2u, symbol Device:L
- added R23: 100k, symbol Device:R_Small
- added R24: 20k, symbol Device:R_Small
- added R25: 135k, symbol Device:R_Small
- added R26: 30k, symbol Device:R_Small
- added U4: TPS566242DRLR, footprints:SOT5x3_DRL_TEX, symbol TPS566242DRLR:TPS566242DRLR
Connections:
- net +3.3V: now also C22.1, C23.1, C24.1, C25.1, C26.1, C27.1, L3.2, R25.1
- net GND: now also C19.2, C20.2, C21.2, C23.2, C24.2, C25.2, C26.2, C27.2, R24.2, R26.2, U4.3 (GND), U4.4 (AGND)
- new net: C22.2, R25.2, R26.1, U4.6 (FB)
- new net +12V: C19.1, C20.1, C21.1, R23.1, U4.1 (VIN)
- new net EN: R23.2, R24.1, U4.5 (EN)
- new net SW: L3.1, U4.2 (SW)
- no-connect marks 2 -> 0

Commit message: feat: added footprints
Parts:
- C19, C20, C21, C22, C23, C24, C25, C26, C27, L3: footprint (none) -> Capacitor_SMD:C_0201_0603Metric_Pad0.64x0.40mm_HandSolder
- R23, R24, R25, R26: footprint (none) -> Resistor_SMD:R_0201_0603Metric_Pad0.64x0.40mm_HandSolder
Changed lines of the file:
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@@
 			)
 		)
-		(property "Footprint" ""
+		(property "Footprint" "Capacitor_SMD:C_0201_0603Metric_Pad0.64x0.40mm_HandSolder"
 			(at 100.33 33.02 0)
 			(effects
@@
 			)
 		)
-		(property "Footprint" ""
+		(property "Footprint" "Capacitor_SMD:C_0201_0603Metric_Pad0.64x0.40mm_HandSolder"
 			(at 147.32 35.56 0)
 			(effects
@@
 			)
 		)
-		(property "Footprint" ""
+		(property "Footprint" "Capacitor_SMD:C_0201_0603Metric_Pad0.64x0.40mm_HandSolder"
 			(at 26.67 38.1 0)
 			(effects
@@
 			)
 		)
-		(property "Footprint" ""
+		(property "Footprint" "Resistor_SMD:R_0201_0603Metric_Pad0.64x0.40mm_HandSolder"
 			(at 44.45 45.72 0)
 			(effects
@@
 			)
 		)
-		(property "Footprint" ""
+		(property "Footprint" "Capacitor_SMD:C_0201_0603Metric_Pad0.64x0.40mm_HandSolder"
 			(at 121.92 35.56 0)
 			(effects
@@
 			)
 		)
-		(property "Footprint" ""
+		(property "Footprint" "Resistor_SMD:R_0201_0603Metric_Pad0.64x0.40mm_HandSolder"
 			(at 44.45 38.1 0)
 			(effects
@@
 			)
 		)
-		(property "Footprint" ""
+		(property "Footprint" "Resistor_SMD:R_0201_0603Metric_Pad0.64x0.40mm_HandSolder"
 			(at 111.76 43.18 0)
 			(effects
@@
 			)
 		)
-		(property "Footprint" ""
+		(property "Footprint" "Capacitor_SMD:C_0201_0603Metric_Pad0.64x0.40mm_HandSolder"
 			(at 104.14 35.56 0)
 			(effects
@@
 			)
 		)
-		(property "Footprint" ""
+		(property "Footprint" "Capacitor_SMD:C_0201_0603Metric_Pad0.64x0.40mm_HandSolder"
 			(at 35.56 38.1 0)
 			(effects
@@
 			)
 		)
-		(property "Footprint" ""
+		(property "Footprint" "Capacitor_SMD:C_0201_0603Metric_Pad0.64x0.40mm_HandSolder"
 			(at 156.21 35.56 0)
 			(effects
@@
 			)
 		)
-		(property "Footprint" ""
+		(property "Footprint" "Capacitor_SMD:C_0201_0603Metric_Pad0.64x0.40mm_HandSolder"
 			(at 17.78 38.1 0)
 			(effects
@@
 			)
 		)
-		(property "Footprint" ""
+		(property "Footprint" "Capacitor_SMD:C_0201_0603Metric_Pad0.64x0.40mm_HandSolder"
 			(at 138.43 35.56 0)
 			(effects
@@
 			)
 		)
-		(property "Footprint" ""
+		(property "Footprint" "Resistor_SMD:R_0201_0603Metric_Pad0.64x0.40mm_HandSolder"
 			(at 111.76 35.56 0)
 			(effects
@@
 			)
 		)
-		(property "Footprint" ""
+		(property "Footprint" "Capacitor_SMD:C_0201_0603Metric_Pad0.64x0.40mm_HandSolder"
 			(at 129.54 35.56 0)
 			(effects
