File: buck12v.kicad_sch (KiCad schematic)
At the start: 11 parts, among them U2 LM76005

Commit message: updates
Connections:
- net V_switched renamed 48v_switched
Changed lines of the file:
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@@
 		)
 	)
-	(global_label "V_switched"
+	(global_label "48v_switched"
 		(shape input)
 		(at 71.12 78.74 180)
@@
 		)
 		(property "Intersheetrefs" "${INTERSHEET_REFS}"
-			(at 57.9143 78.74 0)
+			(at 55.6163 78.74 0)
 			(effects
 				(font

Commit message: Renaming of Parts
Rename
Parts:
- Rfbb1: value 9.09kOhm -> 9.09k
- Rfbt1, Rpgood1: value 100kOhm -> 100k
Changed lines of the file:
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@@
 		(rev "Rev 1.0.0")
 		(company "UMass Robotics")
+		(comment 3 "Alperen Ozpolat")
 		(comment 4 "Niranjan Mathirajan")
 	)
@@
 			)
 		)
-		(property "Value" "100kOhm"
+		(property "Value" "100k"
 			(at 130.556 70.358 90)
 			(effects
@@
 			)
 		)
-		(property "Value" "100kOhm"
+		(property "Value" "100k"
 			(at 190.5 88.646 0)
 			(effects
@@
 			)
 		)
-		(property "Value" "9.09kOhm"
+		(property "Value" "9.09k"
 			(at 190.754 107.696 0)
 			(effects

Commit message: updates
Parts:
- renumbered U2 to U3
Changed lines of the file:
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@@
 		(dnp no)
 		(fields_autoplaced yes)
-		(property "Reference" "#PWR011"
+		(property "Reference" "#PWR022"
 			(at 180.34 93.98 0)
 			(effects
@@
 			(project "doggie_board"
 				(path "/883cb7fa-3eb5-48d4-9cde-7c11307d94f0/ccf07133-5d0c-4081-9a30-ebff06623cf2"
-					(reference "#PWR011")
+					(reference "#PWR022")
 					(unit 1)
 				)
@@
 		(dnp no)
 		(fields_autoplaced yes)
-		(property "Reference" "#PWR013"
+		(property "Reference" "#PWR021"
 			(at 161.29 123.19 0)
 			(effects
@@
 			(project "doggie_board"
 				(path "/883cb7fa-3eb5-48d4-9cde-7c11307d94f0/ccf07133-5d0c-4081-9a30-ebff06623cf2"
-					(reference "#PWR013")
+					(reference "#PWR021")
 					(unit 1)
 				)
@@
 		(dnp no)
 		(fields_autoplaced yes)
-		(property "Reference" "U2"
+		(property "Reference" "U3"
 			(at 146.05 73.66 0)
 			(effects
@@
 			(project "doggie_board"
 				(path "/883cb7fa-3eb5-48d4-9cde-7c11307d94f0/ccf07133-5d0c-4081-9a30-ebff06623cf2"
-					(reference "U2")
+					(reference "U3")
 					(unit 1)
 				)
@@
 		(dnp no)
 		(fields_autoplaced yes)
-		(property "Reference" "#PWR07"
+		(property "Reference" "#PWR023"
 			(at 260.35 83.82 0)
 			(effects
@@
 			(project "doggie_board"
 				(path "/883cb7fa-3eb5-48d4-9cde-7c11307d94f0/ccf07133-5d0c-4081-9a30-ebff06623cf2"
-					(reference "#PWR07")
+					(reference "#PWR023")
 					(unit 1)
 				)
@@
 		(dnp no)
 		(fields_autoplaced yes)
-		(property "Reference" "#FLG03"
+		(property "Reference" "#FLG04"
 			(at 240.03 78.105 0)
 			(effects
@@
 			(project ""
 				(path "/883cb7fa-3eb5-48d4-9cde-7c11307d94f0/ccf07133-5d0c-4081-9a30-ebff06623cf2"
-					(reference "#FLG03")
+					(reference "#FLG04")
 					(unit 1)
 				)
@@
 		(dnp no)
 		(fields_autoplaced yes)
-		(property "Reference" "#PWR014"
+		(property "Reference" "#PWR020"
 			(at 149.86 132.08 0)
 			(effects
@@
 			(project "doggie_board"
 				(path "/883cb7fa-3eb5-48d4-9cde-7c11307d94f0/ccf07133-5d0c-4081-9a30-ebff06623cf2"
-					(reference "#PWR014")
-					(unit 1)
-				)
+					(reference "#PWR020")
+					(unit 1)
+				)

Commit message: fixed ERC
Connections:
- net 48v_switched renamed +48V
Changed lines of the file:
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@@
+	)
+	(junction
+		(at 73.66 78.74)
+		(diameter 0)
+		(color 0 0 0 0)
 	)
 	(junction
@@
 	(wire
 		(pts
-			(xy 71.12 78.74) (xy 92.71 78.74)
+			(xy 71.12 78.74) (xy 73.66 78.74)
 		)
 		(stroke
@@
 	(wire
 		(pts
+			(xy 73.66 78.74) (xy 92.71 78.74)
+		)
+		(stroke
+			(width 0)
+			(type default)
+		)
+	)
+	(wire
+		(pts
 			(xy 118.11 113.03) (xy 118.11 104.14)
 		)
@@
 			(width 0)
 			(type default)
-		)
-	)
-	(global_label "48v_switched"
-		(shape input)
-		(at 71.12 78.74 180)
-		(fields_autoplaced yes)
-		(effects
-			(font
-				(size 1.27 1.27)
-			)
-			(justify right)
-		)
-		(property "Intersheetrefs" "${INTERSHEET_REFS}"
-			(at 55.6163 78.74 0)
-			(effects
-				(font
-					(size 1.27 1.27)
-				)
-				(justify right)
-				(hide yes)
-			)
 		)
 	)
@@
 					(unit 1)
 				)
+			)
+		)
+	)
+	(symbol
+		(lib_id "power:+48V")
+		(at 73.66 78.74 0)
+		(unit 1)
+		(exclude_from_sim no)
+		(in_bom yes)
+		(on_board yes)
+		(dnp no)
+		(fields_autoplaced yes)
+		(property "Reference" "#PWR012"
+			(at 73.66 82.55 0)
+			(effects
+				(font
+					(size 1.27 1.27)
+				)
+				(hide yes)
+			)
+		)
+		(property "Value" "+48V"
+			(at 73.66 73.66 0)
+			(effects
+				(font
+					(size 1.27 1.27)
+				)
+			)
+		)
+		(property "Footprint" ""
+			(at 73.66 78.74 0)
+			(effects
+				(font
+					(size 1.27 1.27)
+				)
+				(hide yes)
+			)
+		)
+		(property "Datasheet" ""
+			(at 73.66 78.74 0)
+			(effects
+				(font
+					(size 1.27 1.27)
+				)
+				(hide yes)
+			)
+		)
+		(property "Description" "Power symbol creates a global label with name \"+48V\""
+			(at 73.66 78.74 0)
+			(effects
+				(font
+					(size 1.27 1.27)
+				)
+				(hide yes)
+			)
+		)
+		(pin "1"
+		)
+		(instances
+			(project "doggie_board"
+				(path "/883cb7fa-3eb5-48d4-9cde-7c11307d94f0/ccf07133-5d0c-4081-9a30-ebff06623cf2"
+					(reference "#PWR012")
+					(unit 1)
+				)

Commit message: Fixed Schematics with more cost effective IC's
Parts:
- removed Cboot1: 470nF, 20mOhm, Capacitor_SMD:C_0805_2012Metric_Pad1.18x1.45mm_HandSolder, symbol Device:C
- removed Cin1: 4.7uF, 5.89mOhm, Capacitor_SMD:C_0805_2012Metric_Pad1.18x1.45mm_HandSolder, symbol Device:C
- removed Cinx1: 470nF, 33.996mOhm, Capacitor_SMD:C_0805_2012Metric_Pad1.18x1.45mm_HandSolder, symbol Device:C
- removed Cout1: 150uF, Capacitor_SMD:C_0805_2012Metric_Pad1.18x1.45mm_HandSolder, symbol Device:C_Polarized_US
- removed Coutx1: 470nF, 87.491mOhm, Capacitor_SMD:C_0805_2012Metric_Pad1.18x1.45mm_HandSolder, symbol Device:C
- removed Cvcc1: 2.2uF, 7.674mOhm, Capacitor_SMD:C_0805_2012Metric_Pad1.18x1.45mm_HandSolder, symbol Device:C
- removed Rfbb1: 9.09k, Resistor_SMD:R_0201_0603Metric, symbol Device:R
- removed Rfbt1, Rpgood1: 100k, Resistor_SMD:R_0201_0603Metric, symbol Device:R
- removed U3: LM76005, Package_DFN_QFN:Texas_RNP0030B_WQFN-30-1EP_4x6mm_P0.5mm_EP1.8x4.5mm_ThermalVias, symbol Regulator_Switching:LM76005
- added C3, C4, C6, C8: 2.2u, symbol Device:C_Small
- added C5: 1.8n, symbol Device:C_Small
- added C7: 47p, symbol Device:C_Small
- added C9: 10u, symbol Device:C_Small
- added Q7, Q8: Q_NMOS, symbol Device:Q_NMOS
- added R13: 24.9k, symbol Device:R
- added R14: 40.2k, symbol Device:R
- added R15: 100k, symbol Device:R
- added R16: 47.5k, symbol Device:R
- added R17: 4.42k, symbol Device:R
- added R18: R, symbol Device:R
- added U2: LM5148RGYR, footprints:QFN50P550X350X100-25N, symbol LM5148:LM5148RGYR
- L1: value 15uH, 16.9mOhm -> L; footprint Inductor_SMD:L_6.3x6.3_H3 -> (none)
Connections:
- net +12V: now also C9.1, R18.2, U2.21 (VOUT); no longer L1.2
- net GND: now also C3.2, C6.2, C7.2, C8.2, C9.2, Q7.S, R13.2, R14.2, R17.2, U2.10 (PGND), U2.16 (VCCX), U2.25 (EP), U2.7 (AGND)
- net at L1.1: now also C4.2, Q7.D, Q8.S, U2.14 (SW)
- new net: R14.1, U2.3 (CNFG)
- new net: C4.1, U2.15 (CBOOT)
- new net: Q7.G, U2.11 (LO)
- new net: C5.1, C7.1, U2.5 (EXTCOMP)
- new net: C5.2, R17.1
- new net: L1.2, R18.1, U2.20 (ISNS+)
- new net: R15.2, U2.17 (PG/SYNCOUT)
- new net: Q8.G, U2.13 (HO)
- new net: R16.2, U2.6 (FB)
- new net 48_RAW: C3.1, Q8.D, U2.12 (VIN), U2.19 (EN)
- new net PFM_SYNC: C6.1, R16.1, U2.18 (PFM/SYNC), U2.8 (VDDA)
- new net RT: R13.1, U2.4 (RT)
- new net VCC: C8.1, R15.1, U2.9 (VCC)
- no-connect marks 2 -> 0

Commit message: feat: added footprints
Parts:
- C3, C4, C5, C6, C7, C8, C9: footprint (none) -> Capacitor_SMD:C_0201_0603Metric_Pad0.64x0.40mm_HandSolder
- L1: value L -> 4.7u
- R13, R14, R15, R16, R17: footprint (none) -> Resistor_SMD:R_0201_0603Metric_Pad0.64x0.40mm_HandSolder
- R18: value R -> 6m
Changed lines of the file:
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@@
 			)
 		)
-		(property "Footprint" ""
+		(property "Footprint" "Resistor_SMD:R_0201_0603Metric_Pad0.64x0.40mm_HandSolder"
 			(at 23.622 40.64 90)
 			(effects
@@
 			)
 		)
-		(property "Footprint" ""
+		(property "Footprint" "Capacitor_SMD:C_0201_0603Metric_Pad0.64x0.40mm_HandSolder"
 			(at 87.63 39.37 0)
 			(effects
@@
 			)
 		)
-		(property "Footprint" ""
+		(property "Footprint" "Capacitor_SMD:C_0201_0603Metric_Pad0.64x0.40mm_HandSolder"
 			(at 148.59 52.07 0)
 			(effects
@@
 			)
 		)
-		(property "Footprint" ""
+		(property "Footprint" "Capacitor_SMD:C_0201_0603Metric_Pad0.64x0.40mm_HandSolder"
 			(at 33.02 19.05 0)
 			(effects
@@
 			)
 		)
-		(property "Footprint" ""
+		(property "Footprint" "Capacitor_SMD:C_0201_0603Metric_Pad0.64x0.40mm_HandSolder"
 			(at 88.9 69.85 0)
 			(effects
@@
 			)
 		)
-		(property "Footprint" ""
+		(property "Footprint" "Resistor_SMD:R_0201_0603Metric_Pad0.64x0.40mm_HandSolder"
 			(at 17.272 21.59 90)
 			(effects
@@
 			)
 		)
-		(property "Footprint" ""
+		(property "Footprint" "Capacitor_SMD:C_0201_0603Metric_Pad0.64x0.40mm_HandSolder"
 			(at 106.68 29.21 0)
 			(effects
@@
 			)
 		)
-		(property "Value" "L"
+		(property "Value" "4.7u"
 			(at 129.54 46.99 90)
 			(effects
@@
 			)
 		)
-		(property "Footprint" ""
+		(property "Footprint" "Resistor_SMD:R_0201_0603Metric_Pad0.64x0.40mm_HandSolder"
 			(at 31.242 58.42 90)
 			(effects
@@
 			)
 		)
-		(property "Value" "R"
+		(property "Value" "6m"
 			(at 139.7 45.72 90)
 			(effects
@@
 			)
 		)
-		(property "Footprint" ""
+		(property "Footprint" "Capacitor_SMD:C_0201_0603Metric_Pad0.64x0.40mm_HandSolder"
 			(at 96.52 31.75 0)
 			(effects
@@
 			)
 		)
-		(property "Footprint" ""
+		(property "Footprint" "Resistor_SMD:R_0201_0603Metric_Pad0.64x0.40mm_HandSolder"
 			(at 38.1 53.848 90)
 			(effects
@@
 			)
 		)
-		(property "Footprint" ""
+		(property "Footprint" "Capacitor_SMD:C_0201_0603Metric_Pad0.64x0.40mm_HandSolder"
 			(at 99.06 73.66 0)
 			(effects
@@
 			)
 		)
-		(property "Footprint" ""
+		(property "Footprint" "Resistor_SMD:R_0201_0603Metric_Pad0.64x0.40mm_HandSolder"
 			(at 87.122 77.47 90)
 			(effects

Commit message: added headers and modified some stuff
Parts:
- added J5, J6: Conn_01x02, symbol Connector_Generic:Conn_01x02
- added Q10: Q_NMOS, symbol Device:Q_NMOS
- R15: value 100k -> 470k; footprint Resistor_SMD:R_0201_0603Metric_Pad0.64x0.40mm_HandSolder -> (none)
Connections:
- net +12V: now also R15.1
- net 48_RAW: now also J5.2 (Pin_2); no longer U2.19 (EN)
- net GND: now also J6.2 (Pin_2), Q10.G
- net VCC: no longer R15.1
- net 12V_PG: now reaches R15.2, U2.17 (PG/SYNCOUT)
- net 12V_PG: now also Q10.D
- net PFM_SYNC renamed VDDA
- new net: J6.1 (Pin_1), Q10.S
- new net: J5.1 (Pin_1), U2.19 (EN)
Other:
- note added: "Bridge to always enable 12V"
- note added: "We add transistor as diode to prevent 12v pullup from messing with 5/3.3V logic Note: Vf is around 1V so it does not get pulled all the way to ground!"
