File: misc.kicad_sch (KiCad schematic)
At the start: 4 parts

Commit message: feat: added footprints
Parts:
- H1, H2, H3, H4: footprint (none) -> MountingHole:MountingHole_5.3mm_M5_DIN965_Pad_TopBottom
Changed lines of the file:
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@@
 			)
 		)
-		(property "Footprint" ""
+		(property "Footprint" "MountingHole:MountingHole_5.3mm_M5_DIN965_Pad_TopBottom"
 			(at 35.56 64.77 0)
 			(effects
@@
 			)
 		)
-		(property "Footprint" ""
+		(property "Footprint" "MountingHole:MountingHole_5.3mm_M5_DIN965_Pad_TopBottom"
 			(at 35.56 50.8 0)
 			(effects
@@
 			)
 		)
-		(property "Footprint" ""
+		(property "Footprint" "MountingHole:MountingHole_5.3mm_M5_DIN965_Pad_TopBottom"
 			(at 59.69 64.77 0)
 			(effects
@@
 			)
 		)
-		(property "Footprint" ""
+		(property "Footprint" "MountingHole:MountingHole_5.3mm_M5_DIN965_Pad_TopBottom"
 			(at 59.69 50.8 0)
 			(effects

Commit message: pcb routing
Parts:
- H1, H2, H3, H4: footprint MountingHole:MountingHole_5.3mm_M5_DIN965_Pad_TopBottom -> MountingHole:MountingHole_3.2mm_M3_DIN965_Pad_TopBottom

Commit message: updated headers
Parts:
- added R19: 270k, Resistor_SMD:R_0603_1608Metric_Pad0.98x0.95mm_HandSolder, symbol Device:R_Small
- added R20: 20k, Resistor_SMD:R_0603_1608Metric_Pad0.98x0.95mm_HandSolder, symbol Device:R_Small
Connections:
- net 48_RAW: now also R19.1
- net GND: now also R20.2
- new net +3.3V_LP: R19.2, R20.1
